File: Motherboard/motherboard_2022_2023/motherboard_2022_2023.kicad_sch (KiCad schematic)
At the start: 12 parts, among them J1 Conn_01x02_Female, J2 Raspberry_Pi_2_3, U1 XBee_THT, U2 PCA9685PW

Commit message: Add 2 pyro channels
Parts:
- J10: renamed from J?; footprint custom-footprints:XBee-THT -> Connector_PinHeader_2.54mm:PinHeader_1x03_P2.54mm_Vertical
- J2: footprint (none) -> Connector_PinHeader_2.54mm:PinHeader_2x20_P2.54mm_Vertical
- J3, J4, J5, J6, J7, J8, J9: renamed from J?; footprint (none) -> Connector_PinHeader_2.54mm:PinHeader_1x03_P2.54mm_Vertical
- U1: footprint (none) -> custom-footprints:XBee-THT
Other:
- added sheet Pyro Channel Pair (pyro_channel_pair.kicad_sch)

Commit message: Preliminary PCB layout
Parts:
- J2: footprint Connector_PinHeader_2.54mm:PinHeader_2x20_P2.54mm_Vertical -> custom-footprints:PI_Zero
Changed lines of the file:
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@@
       (effects (font (size 1.27 1.27)) (justify left))
     )
-    (property "Footprint" "Connector_PinHeader_2.54mm:PinHeader_2x20_P2.54mm_Vertical" (id 2) (at 66.04 91.44 0)
+    (property "Footprint" "custom-footprints:PI_Zero" (id 2) (at 66.04 91.44 0)
       (effects (font (size 1.27 1.27)) hide)
     )
@@
     )
     (path "/0903351d-a664-4c13-a4cb-34445cc34adb"
-      (reference "J2") (unit 1) (value "Raspberry_Pi_2_3") (footprint "Connector_PinHeader_2.54mm:PinHeader_2x20_P2.54mm_Vertical")
+      (reference "J2") (unit 1) (value "Raspberry_Pi_2_3") (footprint "custom-footprints:PI_Zero")
     )
     (path "/0e8a3700-fd0c-4a9f-8839-ef0ab0f24625"

Commit message: Layout pyro channels
Connections:
- net PYRO_B: now reaches U2.15 (LED8)
- net PYRO_A: now reaches U2.16 (LED9)
- net On-Board-Regulation/V_BAT renamed +BATT
- no-connect marks 9 -> 7
Other:
- moved on the sheet: U2

Commit message: Added Dummy Sensors
Parts:
- added U?: MPL3115A2, Package_LGA:NXP_LGA-8_3x5mm_P1.25mm_H1.1mm, symbol Sensor_Pressure:MPL3115A2
- added U?: BNO055, Package_LGA:LGA-28_5.2x3.8mm_P0.5mm, symbol Sensor_Motion:BNO055
Connections:
- net +5V: now also U?.1 (VDD), U?.3 (VDD)
- net GND: now also U?.2 (GND), U?.3 (GND)
- new net: U?.15 (GNDIO), U?.16 (GNDIO), U?.25 (GNDIO)
Other:
- moved on the sheet: J1

Commit message: Added SDA/SCL & Document Titles
Parts:
- added R1, R2: 100k, symbol Device:R
- gave numbers to parts that had none: 2
- renumbered U2 to U3
Connections:
- net +3V3: now also U2.28 (VDDIO), U2.3 (VDD), R1.1, R2.1
- net +5V: no longer U2.3 (VDD)
- net SCL: now also U2.19 (COM1), U4.7 (SDL), R2.2
- net SDA: now also U2.20 (COM0), U4.8 (SCL), R1.2
- no-connect marks 7 -> 8

Commit message: Add SAM-M8Q
Parts:
- added D?: Yellow, symbol Device:LED_Small
- added R?: 1k, symbol Device:R_Small
- added TP? (x2): TestPoint, symbol Connector:TestPoint
- added U?: SAM-M8Q, RF_GPS:ublox_SAM-M8Q, symbol RF_GPS:SAM-M8Q
Connections:
- net +3V3: now also U?.17 (VCC), U?.2 (VCC_IO), U?.3 (V_BCKP)
- net GND: now also D?.1 (K), U?.1 (GND), U?.10 (GND), U?.11 (GND), U?.15 (GND), U?.16 (GND), U?.20 (GND), U?.4 (GND), U?.5 (GND), U?.6 (GND)
- net SCL: now also U?.12 (SCL)
- net SDA: now also U?.9 (SDA)
- new net: TP?.1, U?.13 (TXD)
- new net: TP?.1, U?.14 (RXD)
- new net: D?.2 (A), R?.2
- new net PPS: R?.1, U?.7 (TIMEPULSE)
- no-connect marks 8 -> 11
Other:
- note added: "Can be used for RTC backup, investigate"
- moved on the sheet: U2, U4

Commit message: Nuked BNO055 & Re Laid Out Schematic
Parts:
- removed U2: BNO055, Package_LGA:LGA-28_5.2x3.8mm_P0.5mm, symbol Sensor_Motion:BNO055
- R1, R2: value 100k -> 10k
Connections:
- no-connect marks 11 -> 10
Other:
- moved on the sheet: D?, R?, TP?, U4, U?

Commit message: New MPU6050 Symbol
Parts:
- added JP?: SolderJumper_3_Bridged12, symbol Jumper:SolderJumper_3_Bridged12
- added R?: 100k, symbol Device:R
- added U?: MPU-6050, Connector_PinSocket_2.54mm:PinSocket_1x08_P2.54mm_Vertical, symbol custom_symbols:MPU-6050
Connections:
- net +5V: now also U?.1 (VCC)
- net GND: now also R?.1, U?.2 (GND)
- net SCL: now also U?.3 (SCL)
- net SDA: now also U?.4 (SDA)
- new net: JP?.1 (A), R?.2
- new net: JP?.2 (C), U?.7 (ADD)
