File: Motherboard/motherboard_2022_2023/motherboard_2022_2023.kicad_sch (KiCad schematic)
At the start: 26 parts, among them J1 Conn_01x02_Female, J10 Conn_01x03_Male, J2 Raspberry_Pi_2_3, J3 Conn_01x03_Male, J4 Conn_01x03_Male, J5 Conn_01x03_Male, J6 Conn_01x03_Male, J7 Conn_01x03_Male, J8 Conn_01x03_Male, J9 Conn_01x03_Male, U1 XBee_THT, U2 MPU-6050-Breakout, U3 PCA9685PW, U4 MPL3115A2, U6 SAM-M8Q

Commit message: Another Buzzer Option
Parts:
- BZ1: footprint custom-footprints:8RT1209P-C -> custom-footprints:CPI-1375-80T
Changed lines of the file:
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@@
       (effects (font (size 1.27 1.27)) (justify left))
     )
-    (property "Footprint" "custom-footprints:8RT1209P-C" (id 2) (at 135.255 149.86 90)
+    (property "Footprint" "custom-footprints:CPI-1375-80T" (id 2) (at 135.255 149.86 90)
       (effects (font (size 1.27 1.27)) hide)
     )
@@
     )
     (path "/dce5d536-e66b-40aa-9add-0f38dedf7b75"
-      (reference "BZ1") (unit 1) (value "Buzzer") (footprint "custom-footprints:8RT1209P-C")
+      (reference "BZ1") (unit 1) (value "Buzzer") (footprint "custom-footprints:CPI-1375-80T")
     )
     (path "/e3dd2361-8a26-4d67-8fa2-04aedf170f2c/2858d813-a628-43ec-b026-ff8014913678"

Commit message: Add option to use standalone MPU-6050 chip Also corrects a couple small bugs in footprints
Parts:
- added C6, C9: 100n, Capacitor_SMD:C_0603_1608Metric, symbol Device:C_Small
- added C7: 10n, Capacitor_SMD:C_0603_1608Metric, symbol Device:C_Small
- added C8: 2.2n, Capacitor_SMD:C_0603_1608Metric, symbol Device:C_Small
- added U7: MPU-6050, Sensor_Motion:InvenSense_QFN-24_4x4mm_P0.5mm, symbol Sensor_Motion:MPU-6050
Connections:
- net +3V3: now also C6.2, C7.2, U7.13 (VDD), U7.8 (VDDIO)
- net GND: now also C6.1, C7.1, C8.2, C9.2, U7.1 (CLKIN), U7.11 (FSYNC), U7.18 (GND), U7.9 (AD0)
- net SCL: now also U7.24 (SDA)
- net SDA: now also U7.23 (SCL)
- new net: C9.1, U7.10 (REGOUT)
- new net: C8.1, U7.20 (CPOUT)
- no-connect marks 13 -> 16
Other:
- moved on the sheet: BZ1

Commit message: Add capacitors to MPL3115 according to the datasheet
Parts:
- added C10, C12: 100n, Capacitor_SMD:C_0603_1608Metric, symbol Device:C_Small
- added C11: 10u, Capacitor_SMD:C_0603_1608Metric, symbol Device:C_Small
- JP3: value SolderJumper_3_Bridged12 -> ADD
Connections:
- net +3V3: now also U4.1 (VDD), U4.4 (VDDIO), C10.2, C11.2
- net +5V: no longer U4.1 (VDD)
- net GND: now also C10.1, C11.1, C12.2
- net at U4.2 (CAP): now also C12.1
- no-connect marks 16 -> 18
Other:
- moved on the sheet: U4

Commit message: Add notes to schematic
Other:
- note added: "TODO: Leaving these floating is a bad idea"
- note removed: "Can be used for RTC backup, investigate"
Changed lines of the file:
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@@
     )
   )
-  (text "Can be used for RTC\nbackup, investigate" (at 250.19 105.41 0)
+  (text "TODO: Leaving these\nfloating is a bad idea" (at 214.63 111.76 0)
     (effects (font (size 1.27 1.27)) (justify left bottom))
   )

Commit message: Connect XBee CTS to pi
Connections:
- net XBEE_UART_~{CTS}: now also J2.36 (GPIO16)
- net XBEE_UART_~{RTS}: now also J2.11 (GPIO17); no longer U1.16 (DIO6/~{RTS})
- no-connect marks 18 -> 21
Other:
- note added: "TODO: Can we safely leave reset, sleep, etc... floating?"
Changed lines of the file:
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@@
   )
   (no_connect (at 149.86 165.1))
+  (no_connect (at 86.36 68.58))
   (no_connect (at 210.82 68.58))
   (no_connect (at 139.7 109.22))
   (no_connect (at 139.7 114.3))
   (no_connect (at 139.7 116.84))
+  (no_connect (at 86.36 71.12))
   (no_connect (at 233.68 121.92))
   (no_connect (at 199.39 118.11))
@@
   (no_connect (at 149.86 160.02))
   (no_connect (at 199.39 115.57))
+  (no_connect (at 86.36 109.22))
   (no_connect (at 175.26 35.56))
   (no_connect (at 210.82 58.42))
@@
     (stroke (width 0) (type default) (color 0 0 0 0))
   )
+  (wire (pts (xy 27.94 76.2) (xy 45.72 76.2))
+    (stroke (width 0) (type default) (color 0 0 0 0))
+  )
   (wire (pts (xy 176.53 147.32) (xy 180.34 147.32))
     (stroke (width 0) (type default) (color 0 0 0 0))
@@
     (stroke (width 0) (type default) (color 0 0 0 0))
   )
-  (wire (pts (xy 17.78 156.21) (xy 35.56 156.21))
-    (stroke (width 0) (type default) (color 0 0 0 0))
-  )
   (wire (pts (xy 111.76 114.3) (xy 121.92 114.3))
     (stroke (width 0) (type default) (color 0 0 0 0))
@@
   )
   (wire (pts (xy 250.19 52.07) (xy 259.08 52.07))
+    (stroke (width 0) (type default) (color 0 0 0 0))
+  )
+  (wire (pts (xy 27.94 78.74) (xy 45.72 78.74))
     (stroke (width 0) (type default) (color 0 0 0 0))
   )
@@
     )
   )
+  (text "TODO: Can we safely leave\nreset, sleep, etc... floating?"
+    (at 30.48 142.24 0)
+    (effects (font (size 1.27 1.27)) (justify left bottom))
+  )
   (text "TODO: Leaving these\nfloating is a bad idea" (at 214.63 111.76 0)
     (effects (font (size 1.27 1.27)) (justify left bottom))
@@
     (effects (font (size 1.27 1.27)) (justify left bottom))
   )
+  (label "XBEE_UART_~{CTS}" (at 27.94 76.2 0)
+    (effects (font (size 1.27 1.27)) (justify left bottom))
+  )
   (label "PWM_3" (at 250.19 21.59 0)
     (effects (font (size 1.27 1.27)) (justify left bottom))
@@
     (effects (font (size 1.27 1.27)) (justify left bottom))
   )
-  (label "XBEE_UART_~{RTS}" (at 17.78 156.21 0)
-    (effects (font (size 1.27 1.27)) (justify left bottom))
-  )
   (label "PWM_2" (at 250.19 74.93 0)
     (effects (font (size 1.27 1.27)) (justify left bottom))
@@
     (effects (font (size 1.27 1.27)) (justify left bottom))
   )
+  (label "XBEE_UART_~{RTS}" (at 27.94 78.74 0)
+    (effects (font (size 1.27 1.27)) (justify left bottom))
+  )

Commit message: Add note to schematic
Connections:
- no-connect marks 21 -> 22
Other:
- note added: "The RTS signal is not needed as the Pi has plenty of buffer and the XBee always asserts CTS regardless of the RTS state"
Changed lines of the file:
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@@
   (no_connect (at 149.86 160.02))
   (no_connect (at 199.39 115.57))
+  (no_connect (at 35.56 156.21))
   (no_connect (at 86.36 109.22))
   (no_connect (at 175.26 35.56))
@@
   )
   (text "TODO: Can we safely leave\nreset, sleep, etc... floating?"
-    (at 30.48 142.24 0)
+    (at 76.2 142.24 0)
     (effects (font (size 1.27 1.27)) (justify left bottom))
   )
+  (text "The RTS signal is not needed\nas the Pi has plenty of buffer\nand the XBee always asserts CTS\nregardless of the RTS state"
+    (at 16.51 143.51 0)
+    (effects (font (size 1.27 1.27)) (justify left bottom))
+  )

Commit message: Revert "Merge branch 'main' of https://github.com/Rose-Rocketry/NASA-USLI-2023-Electrical-Payload"
This reverts commit 2c693e8b656697acdd5394412e94d16fb74b389e, reversing
changes made to c3e2ab575912267e277cfde858d4ce401414edea.
Connections:
- net XBEE_UART_~{CTS}: no longer J2.36 (GPIO16)
- net XBEE_UART_~{RTS}: now also U1.16 (DIO6/~{RTS}); no longer J2.11 (GPIO17)
- no-connect marks 22 -> 18
Other:
- note removed: "TODO: Can we safely leave reset, sleep, etc... floating?"
- note removed: "The RTS signal is not needed as the Pi has plenty of buffer and the XBee always asserts CTS regardless of the RTS state"
Changed lines of the file:
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@@
   )
   (no_connect (at 149.86 165.1))
-  (no_connect (at 86.36 68.58))
   (no_connect (at 210.82 68.58))
   (no_connect (at 139.7 109.22))
   (no_connect (at 139.7 114.3))
   (no_connect (at 139.7 116.84))
-  (no_connect (at 86.36 71.12))
   (no_connect (at 233.68 121.92))
   (no_connect (at 199.39 118.11))
@@
   (no_connect (at 149.86 160.02))
   (no_connect (at 199.39 115.57))
-  (no_connect (at 35.56 156.21))
-  (no_connect (at 86.36 109.22))
   (no_connect (at 175.26 35.56))
   (no_connect (at 210.82 58.42))
@@
     (stroke (width 0) (type default) (color 0 0 0 0))
   )
-  (wire (pts (xy 27.94 76.2) (xy 45.72 76.2))
-    (stroke (width 0) (type default) (color 0 0 0 0))
-  )
   (wire (pts (xy 176.53 147.32) (xy 180.34 147.32))
     (stroke (width 0) (type default) (color 0 0 0 0))
@@
     (stroke (width 0) (type default) (color 0 0 0 0))
   )
+  (wire (pts (xy 17.78 156.21) (xy 35.56 156.21))
+    (stroke (width 0) (type default) (color 0 0 0 0))
+  )
   (wire (pts (xy 111.76 114.3) (xy 121.92 114.3))
     (stroke (width 0) (type default) (color 0 0 0 0))
@@
   )
   (wire (pts (xy 250.19 52.07) (xy 259.08 52.07))
-    (stroke (width 0) (type default) (color 0 0 0 0))
-  )
-  (wire (pts (xy 27.94 78.74) (xy 45.72 78.74))
     (stroke (width 0) (type default) (color 0 0 0 0))
   )
@@
     )
   )
-  (text "TODO: Can we safely leave\nreset, sleep, etc... floating?"
-    (at 76.2 142.24 0)
-    (effects (font (size 1.27 1.27)) (justify left bottom))
-  )
-  (text "The RTS signal is not needed\nas the Pi has plenty of buffer\nand the XBee always asserts CTS\nregardless of the RTS state"
-    (at 16.51 143.51 0)
-    (effects (font (size 1.27 1.27)) (justify left bottom))
-  )
   (text "TODO: Leaving these\nfloating is a bad idea" (at 214.63 111.76 0)
     (effects (font (size 1.27 1.27)) (justify left bottom))
@@
     (effects (font (size 1.27 1.27)) (justify left bottom))
   )
-  (label "XBEE_UART_~{CTS}" (at 27.94 76.2 0)
-    (effects (font (size 1.27 1.27)) (justify left bottom))
-  )
   (label "PWM_3" (at 250.19 21.59 0)
     (effects (font (size 1.27 1.27)) (justify left bottom))
@@
     (effects (font (size 1.27 1.27)) (justify left bottom))
   )
+  (label "XBEE_UART_~{RTS}" (at 17.78 156.21 0)
+    (effects (font (size 1.27 1.27)) (justify left bottom))
+  )
   (label "PWM_2" (at 250.19 74.93 0)
     (effects (font (size 1.27 1.27)) (justify left bottom))
@@
     (effects (font (size 1.27 1.27)) (justify left bottom))
   )
-  (label "XBEE_UART_~{RTS}" (at 27.94 78.74 0)
-    (effects (font (size 1.27 1.27)) (justify left bottom))
-  )

Commit message: Tie pins high
Connections:
- net +3V3: now also U6.18 (~{RESET}), U6.8 (~{SAFEBOOT})
- no-connect marks 18 -> 16
Changed lines of the file:
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@@
   (junction (at 241.3 34.29) (diameter 0) (color 0 0 0 0)
   )
+  (junction (at 231.14 121.92) (diameter 0) (color 0 0 0 0)
+  )
   (junction (at 241.3 26.67) (diameter 0) (color 0 0 0 0)
   )
@@
   (no_connect (at 139.7 114.3))
   (no_connect (at 139.7 116.84))
-  (no_connect (at 233.68 121.92))
   (no_connect (at 199.39 118.11))
-  (no_connect (at 233.68 119.38))
   (no_connect (at 210.82 63.5))
   (no_connect (at 233.68 114.3))
@@
     (stroke (width 0) (type default) (color 0 0 0 0))
   )
+  (wire (pts (xy 229.87 121.92) (xy 231.14 121.92))
+    (stroke (width 0) (type default) (color 0 0 0 0))
+  )
   (wire (pts (xy 189.23 104.14) (xy 189.23 105.41))
     (stroke (width 0) (type default) (color 0 0 0 0))
@@
     (stroke (width 0) (type default) (color 0 0 0 0))
   )
+  (wire (pts (xy 231.14 119.38) (xy 233.68 119.38))
+    (stroke (width 0) (type default) (color 0 0 0 0))
+  )
   (wire (pts (xy 259.08 119.38) (xy 266.7 119.38))
     (stroke (width 0) (type default) (color 0 0 0 0))
@@
     (stroke (width 0) (type default) (color 0 0 0 0))
   )
+  (wire (pts (xy 231.14 121.92) (xy 231.14 119.38))
+    (stroke (width 0) (type default) (color 0 0 0 0))
+  )
   (wire (pts (xy 241.3 57.15) (xy 241.3 49.53))
     (stroke (width 0) (type default) (color 0 0 0 0))
@@
     (stroke (width 0) (type default) (color 0 0 0 0))
   )
+  (wire (pts (xy 231.14 121.92) (xy 233.68 121.92))
+    (stroke (width 0) (type default) (color 0 0 0 0))
+  )
   (wire (pts (xy 210.82 40.64) (xy 218.44 40.64))
     (stroke (width 0) (type default) (color 0 0 0 0))
@@
     (pin "1")
   )
+  (symbol (lib_id "power:+3V3") (at 229.87 121.92 90) (unit 1)
+    (in_bom yes) (on_board yes)
+    (property "Reference" "#PWR0126" (id 0) (at 233.68 121.92 0)
+      (effects (font (size 1.27 1.27)) hide)
+    )
+    (property "Value" "+3V3" (id 1) (at 220.98 121.92 90)
+      (effects (font (size 1.27 1.27)) (justify right))
+    )
+    (property "Footprint" "" (id 2) (at 229.87 121.92 0)
+      (effects (font (size 1.27 1.27)) hide)
+    )
+    (property "Datasheet" "" (id 3) (at 229.87 121.92 0)
+      (effects (font (size 1.27 1.27)) hide)
+    )
+    (pin "1")
+  )
   (symbol (lib_id "power:GND") (at 162.56 182.88 90) (unit 1)
     (in_bom yes) (on_board yes) (fields_autoplaced)
@@
       (reference "#PWR0125") (unit 1) (value "+3V3") (footprint "")
     )
+    (path "/59ca1811-7110-4efb-847f-6fa7f0bb6790"
+      (reference "#PWR0126") (unit 1) (value "+3V3") (footprint "")
+    )
     (path "/dce5d536-e66b-40aa-9add-0f38dedf7b75"
