File: Motherboard/motherboard_2022_2023/motherboard_2022_2023.kicad_sch (KiCad schematic)
At the start: 34 parts, among them J1 Conn_01x02_Female, J10 Conn_01x03_Male, J2 Raspberry_Pi_2_3, J3 Conn_01x03_Male, J4 Conn_01x03_Male, J5 Conn_01x03_Male, J6 Conn_01x03_Male, J7 Conn_01x03_Male, J8 Conn_01x03_Male, J9 Conn_01x03_Male, U1 XBee_THT, U2 MPU-6050-Breakout, U3 PCA9685PW, U4 MPL3115A2, U6 SAM-M8Q, U7 MPU-6050

Commit message: Add HDMI adaptor
Parts:
- added H5, H6: MountingHole, MountingHole:MountingHole_3.2mm_M3, symbol Mechanical:MountingHole
Other:
- added sheet HDMI CSI Conversion (hdmi.kicad_sch)
- added sheet HDMI CSI Conversion1 (hdmi.kicad_sch)
Changed lines of the file:
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@@
+    )
+  )
+  (symbol (lib_id "Mechanical:MountingHole") (at 227.33 147.32 0) (unit 1)
+    (in_bom yes) (on_board yes) (fields_autoplaced)
+    (property "Reference" "H5" (id 0) (at 224.79 146.0499 0)
+      (effects (font (size 1.27 1.27)) (justify right))
+    )
+    (property "Value" "MountingHole" (id 1) (at 224.79 148.5899 0)
+      (effects (font (size 1.27 1.27)) (justify right))
+    )
+    (property "Footprint" "MountingHole:MountingHole_3.2mm_M3" (id 2) (at 227.33 147.32 0)
+      (effects (font (size 1.27 1.27)) hide)
+    )
+    (property "Datasheet" "~" (id 3) (at 227.33 147.32 0)
+      (effects (font (size 1.27 1.27)) hide)
     )
   )
@@
     )
     (pin "1")
+  )
+  (symbol (lib_id "Mechanical:MountingHole") (at 232.41 147.32 0) (unit 1)
+    (in_bom yes) (on_board yes) (fields_autoplaced)
+    (property "Reference" "H6" (id 0) (at 234.95 146.0499 0)
+      (effects (font (size 1.27 1.27)) (justify left))
+    )
+    (property "Value" "MountingHole" (id 1) (at 234.95 148.5899 0)
+      (effects (font (size 1.27 1.27)) (justify left))
+    )
+    (property "Footprint" "MountingHole:MountingHole_3.2mm_M3" (id 2) (at 232.41 147.32 0)
+      (effects (font (size 1.27 1.27)) hide)
+    )
+    (property "Datasheet" "~" (id 3) (at 232.41 147.32 0)
+      (effects (font (size 1.27 1.27)) hide)
+    )
   )
   (symbol (lib_id "power:+3.3V") (at 193.04 20.32 0) (unit 1)
@@
     )
   )
+  (sheet (at 257.81 153.67) (size 20.32 5.08) (fields_autoplaced)
+    (stroke (width 0.1524) (type solid) (color 0 0 0 0))
+    (fill (color 0 0 0 0.0000))
+    (property "Sheet name" "HDMI CSI Conversion1" (id 0) (at 257.81 152.9584 0)
+      (effects (font (size 1.27 1.27)) (justify left bottom))
+    )
+    (property "Sheet file" "hdmi.kicad_sch" (id 1) (at 257.81 159.3346 0)
+      (effects (font (size 1.27 1.27)) (justify left top))
+    )
+  )
+  (sheet (at 257.81 140.97) (size 20.32 5.08) (fields_autoplaced)
+    (stroke (width 0.1524) (type solid) (color 0 0 0 0))
+    (fill (color 0 0 0 0.0000))
+    (property "Sheet name" "HDMI CSI Conversion" (id 0) (at 257.81 140.2584 0)
+      (effects (font (size 1.27 1.27)) (justify left bottom))
+    )
+    (property "Sheet file" "hdmi.kicad_sch" (id 1) (at 257.81 146.6346 0)
+      (effects (font (size 1.27 1.27)) (justify left top))
+    )
+  )
   (sheet (at 49.53 20.32) (size 21.59 7.62) (fields_autoplaced)
     (stroke (width 0.1524) (type solid) (color 0 0 0 0))
@@
     (path "/e3dd2361-8a26-4d67-8fa2-04aedf170f2c" (page "2"))
     (path "/0dec2096-37b6-40f7-aef8-9fa50e6c5c3f" (page "3"))
+    (path "/d86603e7-9c64-46e4-a723-6cebcaa28a84" (page "4"))
+    (path "/70244b11-01d6-4c0c-a68f-613b116dd32b" (page "5"))
   )
   (symbol_instances
@@
       (reference "C12") (unit 1) (value "100n") (footprint "Capacitor_SMD:C_0603_1608Metric")
     )
+    (path "/0dec2096-37b6-40f7-aef8-9fa50e6c5c3f/f4dc855a-dccd-4c72-b63c-a6ce52f8e549"
+      (reference "D1") (unit 1) (value "3v3") (footprint "")
+    )
     (path "/1e903c2f-be4c-4c28-a5c5-9a13f4e03cde"
       (reference "H1") (unit 1) (value "MountingHole") (footprint "MountingHole:MountingHole_3.2mm_M3")
@@
       (reference "H4") (unit 1) (value "MountingHole") (footprint "MountingHole:MountingHole_3.2mm_M3")
     )
+    (path "/91331a8d-f283-40c1-8ecf-377f52f072ba"
+      (reference "H5") (unit 1) (value "MountingHole") (footprint "MountingHole:MountingHole_3.2mm_M3")
+    )
+    (path "/bec56f43-9891-4854-b3c0-a6dddaf8436b"
+      (reference "H6") (unit 1) (value "MountingHole") (footprint "MountingHole:MountingHole_3.2mm_M3")
+    )
     (path "/ca5c2dbe-aad1-4009-8460-d2c5eb2b32be"
       (reference "J1") (unit 1) (value "Conn_01x02_Female") (footprint "Connector_AMASS:AMASS_XT30PW-M_1x02_P2.50mm_Horizontal")
@@
       (reference "J12") (unit 1) (value "Conn_01x02") (footprint "TerminalBlock_Phoenix:TerminalBlock_Phoenix_PT-1,5-2-5.0-H_1x02_P5.00mm_Horizontal")
     )
+    (path "/d86603e7-9c64-46e4-a723-6cebcaa28a84/eb6c4c24-52d8-4774-90a3-4fe2841ee201"
+      (reference "J13") (unit 1) (value "Conn_01x22_Shielded") (footprint "custom-footprints:MOLEX 22 Pin FPC 54548-2271")
+    )
+    (path "/d86603e7-9c64-46e4-a723-6cebcaa28a84/67bfe331-b0fb-4434-b98d-debe431a46ba"
+      (reference "J14") (unit 1) (value "HDMI_C_1.4") (footprint "custom-footprints:WURTH_685119136923")
+    )
+    (path "/70244b11-01d6-4c0c-a68f-613b116dd32b/eb6c4c24-52d8-4774-90a3-4fe2841ee201"
+      (reference "J15") (unit 1) (value "Conn_01x22_Shielded") (footprint "custom-footprints:MOLEX 22 Pin FPC 54548-2271")
+    )
+    (path "/70244b11-01d6-4c0c-a68f-613b116dd32b/67bfe331-b0fb-4434-b98d-debe431a46ba"
+      (reference "J16") (unit 1) (value "HDMI_C_1.4") (footprint "custom-footprints:WURTH_685119136923")
+    )
     (path "/0dec2096-37b6-40f7-aef8-9fa50e6c5c3f/114ef850-6681-4083-96d2-5c6ecdad19ab"
       (reference "JP1") (unit 1) (value "PYRO_A_SENSE_BYPASS") (footprint "Jumper:SolderJumper-2_P1.3mm_Bridged_RoundedPad1.0x1.5mm")
@@
     )
     (path "/0dec2096-37b6-40f7-aef8-9fa50e6c5c3f/a0c79f21-d2f7-435d-8df3-48bf370d5bc9"
-      (reference "R9") (unit 1) (value "200k") (footprint "Resistor_SMD:R_0603_1608Metric")
+      (reference "R9") (unit 1) (value "100k") (footprint "Resistor_SMD:R_0603_1608Metric")
     )
     (path "/0dec2096-37b6-40f7-aef8-9fa50e6c5c3f/1caf4b80-a97f-49a5-8c39-c7b5b9b741b7"
@@
     )
     (path "/0dec2096-37b6-40f7-aef8-9fa50e6c5c3f/8ef7e272-c64c-4dd6-9dfd-9d3714e220fb"
-      (reference "R11") (unit 1) (value "200k") (footprint "Resistor_SMD:R_0603_1608Metric")
+      (reference "R11") (unit 1) (value "100k") (footprint "Resistor_SMD:R_0603_1608Metric")
     )
     (path "/0dec2096-37b6-40f7-aef8-9fa50e6c5c3f/23a9e7ee-a86a-4c27-9a2f-00d96b6b2cd8"

Commit message: Add mousebite
Connections:
- net PYRO_B_SENSE: now reaches J2.24 (~{CE0}/GPIO8)
- net PYRO_A_SENSE: now reaches J2.26 (~{CE1}/GPIO7)
- no-connect marks 16 -> 48
Other:
- removed sheet HDMI CSI Conversion1
- added sheet HDMI CSI Conversion (reversed) (hdmi 2.kicad_sch)
- moved on the sheet: R1, R2

Commit message: Final Final Adjustments
Parts:
- added C13: 100n, Capacitor_SMD:C_0603_1608Metric, symbol Device:C_Small
- added C14: 10n, Capacitor_SMD:C_0603_1608Metric, symbol Device:C_Small
- TP1: value TestPoint -> RX
- TP2: value TestPoint -> TX
- renumbered J8 to S0, J9 to S1, J10 to S2, J3 to S3, J4 to S4, J5 to S5, J6 to S6, J7 to S7
Connections:
- net +3V3: now also C13.2, C14.2
- net GND: now also C13.1, C14.1

Commit message: Moved CSI to HDMI to own PCB
Other:
- removed sheet HDMI CSI Conversion (reversed)
Changed lines of the file:
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@@
     (pin "3")
-  )
-  (sheet (at 257.81 152.4) (size 20.32 5.08) (fields_autoplaced)
-    (stroke (width 0.1524) (type solid) (color 0 0 0 0))
-    (fill (color 0 0 0 0.0000))
-    (property "Sheet name" "HDMI CSI Conversion (reversed)" (id 0) (at 257.81 151.6884 0)
-      (effects (font (size 1.27 1.27)) (justify left bottom))
-    )
-    (property "Sheet file" "hdmi 2.kicad_sch" (id 1) (at 257.81 158.0646 0)
-      (effects (font (size 1.27 1.27)) (justify left top))
-    )
   )
   (sheet (at 116.84 41.91) (size 21.59 16.51) (fields_autoplaced)
@@
     (path "/0dec2096-37b6-40f7-aef8-9fa50e6c5c3f" (page "3"))
     (path "/d86603e7-9c64-46e4-a723-6cebcaa28a84" (page "4"))
-    (path "/03d26546-991a-429c-b4de-44c077c82641" (page "5"))
   )
   (symbol_instances
@@
       (reference "H6") (unit 1) (value "MountingHole") (footprint "MountingHole:MountingHole_3.2mm_M3")
     )
-    (path "/03d26546-991a-429c-b4de-44c077c82641/bc950924-1296-4adb-a209-9b9be0edae2e"
-      (reference "H7") (unit 1) (value "MountingHole") (footprint "custom-footprints:mousebite")
-    )
     (path "/ca5c2dbe-aad1-4009-8460-d2c5eb2b32be"
       (reference "J1") (unit 1) (value "Conn_01x02_Female") (footprint "Connector_AMASS:AMASS_XT30PW-M_1x02_P2.50mm_Horizontal")
@@
       (reference "J14") (unit 1) (value "HDMI_C_1.4") (footprint "custom-footprints:WURTH_685119136923")
     )
-    (path "/03d26546-991a-429c-b4de-44c077c82641/e046bb90-a8e9-4e7f-8aa0-c8908f4f92d0"
-      (reference "J15") (unit 1) (value "Conn_01x22_Shielded") (footprint "custom-footprints:MOLEX 22 Pin FPC 54548-2271")
-    )
-    (path "/03d26546-991a-429c-b4de-44c077c82641/1cd00081-e313-451c-acb4-77e1c887fa82"
-      (reference "J16") (unit 1) (value "HDMI_C_1.4") (footprint "custom-footprints:WURTH_685119136923")
-    )
     (path "/0dec2096-37b6-40f7-aef8-9fa50e6c5c3f/114ef850-6681-4083-96d2-5c6ecdad19ab"

Commit message: Add ADC
Parts:
- removed H5, H6: MountingHole, MountingHole:MountingHole_3.2mm_M3, symbol Mechanical:MountingHole
- added C15: 10n, Capacitor_SMD:C_0603_1608Metric, symbol Device:C_Small
- added R16: 27k, Resistor_SMD:R_0603_1608Metric, symbol Device:R
- added R17: 10k, Resistor_SMD:R_0603_1608Metric, symbol Device:R
- added U8: MCP3004, Package_SO:SOIC-14_3.9x8.7mm_P1.27mm, symbol Analog_ADC:MCP3004
Connections:
- net +3V3: now also C15.2, U8.13 (Vref), U8.14 (Vdd)
- net +BATT: now also R16.2
- net GND: now also C15.1, R17.1, U8.12 (AGND), U8.7 (DGND)
- net PPS: now also J2.16 (GPIO23); no longer J2.12 (GPIO18/PWM0)
- net MISO: now reaches J2.35 (GPIO19/MISO1)
- net MISO: now also U8.10 (Dout)
- net MCP_CS: now reaches J2.36 (GPIO16)
- net MCP_CS: now also U8.8 (~{CS}/SHDN)
- net MOSI: now reaches J2.38 (GPIO20/MOSI1)
- net MOSI: now also U8.9 (Din)
- net SCLK: now reaches J2.40 (GPIO21/SCLK1)
- net SCLK: now also U8.11 (CLK)
- new net: R16.1, R17.2, U8.1 (CH0)
- no-connect marks 48 -> 47

Commit message: Fix XBee CTS
Connections:
- net XBEE_UART_~{CTS}: now also J2.19 (MOSI0/GPIO10)
- no-connect marks 47 -> 46
Changed lines of the file:
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@@
   (no_connect (at 86.36 88.9))
   (no_connect (at 86.36 99.06))
-  (no_connect (at 86.36 101.6))
   (no_connect (at 86.36 104.14))
   (no_connect (at 86.36 109.22))
@@
   )
   (wire (pts (xy 86.36 111.76) (xy 95.25 111.76))
+    (stroke (width 0) (type default) (color 0 0 0 0))
+  )
+  (wire (pts (xy 86.36 101.6) (xy 102.87 101.6))
     (stroke (width 0) (type default) (color 0 0 0 0))
   )
@@
     (effects (font (size 1.27 1.27)) (justify left bottom))
   )
+  (label "XBEE_UART_~{CTS}" (at 102.87 101.6 180)
+    (effects (font (size 1.27 1.27)) (justify right bottom))
+  )
   (label "MCP_CS" (at 36.83 76.2 0)

Commit message: Remove unneeded I2C pullup resistors The pi zero 2 W already has 1.8k pullups on the board
Parts:
- removed R1, R2: 10k, Resistor_SMD:R_0603_1608Metric, symbol Device:R
Changed lines of the file:
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@@
   (junction (at 58.42 125.73) (diameter 0) (color 0 0 0 0)
   )
-  (junction (at 162.56 91.44) (diameter 0) (color 0 0 0 0)
-  )
   (junction (at 68.58 125.73) (diameter 0) (color 0 0 0 0)
   )
@@
     (stroke (width 0) (type default) (color 0 0 0 0))
   )
-  (wire (pts (xy 162.56 91.44) (xy 162.56 100.33))
-    (stroke (width 0) (type default) (color 0 0 0 0))
-  )
   (wire (pts (xy 259.08 111.76) (xy 261.62 111.76))
     (stroke (width 0) (type default) (color 0 0 0 0))
@@
     (stroke (width 0) (type default) (color 0 0 0 0))
   )
-  (wire (pts (xy 172.72 81.28) (xy 172.72 91.44))
-    (stroke (width 0) (type default) (color 0 0 0 0))
-  )
   (wire (pts (xy 224.79 116.84) (xy 233.68 116.84))
     (stroke (width 0) (type default) (color 0 0 0 0))
@@
     (stroke (width 0) (type default) (color 0 0 0 0))
   )
-  (wire (pts (xy 162.56 91.44) (xy 165.1 91.44))
-    (stroke (width 0) (type default) (color 0 0 0 0))
-  )
   (wire (pts (xy 140.97 39.37) (xy 157.48 39.37))
     (stroke (width 0) (type default) (color 0 0 0 0))
   )
-  (wire (pts (xy 162.56 100.33) (xy 165.1 100.33))
-    (stroke (width 0) (type default) (color 0 0 0 0))
-  )
   (wire (pts (xy 259.08 80.01) (xy 241.3 80.01))
     (stroke (width 0) (type default) (color 0 0 0 0))
@@
     (stroke (width 0) (type default) (color 0 0 0 0))
   )
-  (wire (pts (xy 175.26 81.28) (xy 175.26 100.33))
-    (stroke (width 0) (type default) (color 0 0 0 0))
-  )
   (wire (pts (xy 130.81 99.06) (xy 130.81 104.14))
     (stroke (width 0) (type default) (color 0 0 0 0))
@@
     (stroke (width 0) (type default) (color 0 0 0 0))
   )
-  (wire (pts (xy 162.56 87.63) (xy 162.56 91.44))
-    (stroke (width 0) (type default) (color 0 0 0 0))
-  )
   (wire (pts (xy 60.96 125.73) (xy 63.5 125.73))
     (stroke (width 0) (type default) (color 0 0 0 0))
@@
     (stroke (width 0) (type default) (color 0 0 0 0))
   )
-  (wire (pts (xy 175.26 100.33) (xy 172.72 100.33))
-    (stroke (width 0) (type default) (color 0 0 0 0))
-  )
   (image (at 278.13 175.26) (scale 0.0693664)
     (data
@@
     (effects (font (size 1.27 1.27)) (justify right bottom))
   )
-  (label "SCL" (at 175.26 81.28 270)
-    (effects (font (size 1.27 1.27)) (justify right bottom))
-  )
   (label "SDA" (at 96.52 76.2 180)
     (effects (font (size 1.27 1.27)) (justify right bottom))
@@
     (effects (font (size 1.27 1.27)) (justify left bottom))
   )
-  (label "SDA" (at 172.72 81.28 270)
-    (effects (font (size 1.27 1.27)) (justify right bottom))
-  )
   (label "PWM_6" (at 218.44 45.72 180)
     (effects (font (size 1.27 1.27)) (justify right bottom))
@@
     (pin "3")
   )
-  (symbol (lib_id "power:+3V3") (at 162.56 87.63 0) (unit 1)
-    (in_bom yes) (on_board yes) (fields_autoplaced)
-    (property "Reference" "#PWR09" (id 0) (at 162.56 91.44 0)
-      (effects (font (size 1.27 1.27)) hide)
-    )
-    (property "Value" "+3V3" (id 1) (at 162.56 82.55 0))
-    (property "Footprint" "" (id 2) (at 162.56 87.63 0)
-      (effects (font (size 1.27 1.27)) hide)
-    )
-    (property "Datasheet" "" (id 3) (at 162.56 87.63 0)
-      (effects (font (size 1.27 1.27)) hide)
-    )
-    (pin "1")
-  )
   (symbol (lib_id "power:GND") (at 114.3 52.07 180) (unit 1)
     (in_bom yes) (on_board yes) (fields_autoplaced)
@@
     (pin "1")
   )
-  (symbol (lib_id "Device:R") (at 168.91 91.44 90) (unit 1)
-    (in_bom yes) (on_board yes) (fields_autoplaced)
-    (property "Reference" "R1" (id 0) (at 168.91 85.09 90))
-    (property "Value" "10k" (id 1) (at 168.91 87.63 90))
-    (property "Footprint" "Resistor_SMD:R_0603_1608Metric" (id 2) (at 168.91 93.218 90)
-      (effects (font (size 1.27 1.27)) hide)
-    )
-    (property "Datasheet" "~" (id 3) (at 168.91 91.44 0)
-      (effects (font (size 1.27 1.27)) hide)
-    )
-    (pin "1")
-    (pin "2")
-  )
   (symbol (lib_id "power:+3V3") (at 243.84 101.6 0) (unit 1)
     (in_bom yes) (on_board yes) (fields_autoplaced)
@@
     (pin "1")
   )
-  (symbol (lib_id "Device:R") (at 168.91 100.33 90) (unit 1)
-    (in_bom yes) (on_board yes) (fields_autoplaced)
-    (property "Reference" "R2" (id 0) (at 168.91 93.98 90))
-    (property "Value" "10k" (id 1) (at 168.91 96.52 90))
-    (property "Footprint" "Resistor_SMD:R_0603_1608Metric" (id 2) (at 168.91 102.108 90)
-      (effects (font (size 1.27 1.27)) hide)
-    )
-    (property "Datasheet" "~" (id 3) (at 168.91 100.33 0)
-      (effects (font (size 1.27 1.27)) hide)
-    )
-    (pin "1")
-    (pin "2")
-  )
   (symbol (lib_id "Sensor_Motion:MPU-6050") (at 132.08 167.64 0) (unit 1)
     (in_bom yes) (on_board yes) (fields_autoplaced)
@@
       (reference "#PWR08") (unit 1) (value "+BATT") (footprint "")
     )
-    (path "/33206b03-447c-4b76-a219-a5e499bb1ad2"
-      (reference "#PWR09") (unit 1) (value "+3V3") (footprint "")
-    )
     (path "/135e067f-fb37-40af-88f7-427c16675d5c"
       (reference "#PWR012") (unit 1) (value "GND") (footprint "")
@@
       (reference "Q1") (unit 2) (value "AO4838") (footprint "Package_SO:SOIC-8_3.9x4.9mm_P1.27mm")
     )
-    (path "/42dca09f-ff0a-4405-bf07-04cc646f7d84"
-      (reference "R1") (unit 1) (value "10k") (footprint "Resistor_SMD:R_0603_1608Metric")
-    )
-    (path "/c1f84063-0b2f-4a8e-b53d-51f7366937dc"
-      (reference "R2") (unit 1) (value "10k") (footprint "Resistor_SMD:R_0603_1608Metric")
-    )
     (path "/e3dd2361-8a26-4d67-8fa2-04aedf170f2c/13c198e3-2d63-467b-8892-241e6450945b"
