File: Motherboard/motherboard_2022_2023/motherboard_2022_2023.kicad_sch (KiCad schematic)
At the start: 38 parts, among them J1 Conn_01x02_Female, J2 Raspberry_Pi_2_3, U1 XBee_THT, U2 MPU-6050-Breakout, U3 PCA9685PW, U4 MPL3115A2, U6 SAM-M8Q, U7 MPU-6050, U8 MCP3004

Commit message: Add power switch
Parts:
- added R1: 10k, Resistor_SMD:R_0603_1608Metric, symbol Device:R
- added SW1: SHUTDOWN, Connector_PinHeader_2.54mm:PinHeader_1x02_P2.54mm_Horizontal, symbol Switch:SW_SPST
Connections:
- net +3V3: now also R1.2
- net GND: now also SW1.2 (B)
- net SHUTDOWN: now reaches J2.7 (GCLK0/GPIO4)
- net SHUTDOWN: now also R1.1, SW1.1 (A)
- no-connect marks 46 -> 45
Changed lines of the file:
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@@
   (junction (at 246.38 31.75) (diameter 0) (color 0 0 0 0)
   )
+  (junction (at 166.37 86.36) (diameter 0) (color 0 0 0 0)
+  )
   (junction (at 161.29 60.96) (diameter 0) (color 0 0 0 0)
   )
@@
   (no_connect (at 199.39 118.11))
   (no_connect (at 86.36 71.12))
-  (no_connect (at 86.36 83.82))
   (no_connect (at 86.36 86.36))
   (no_connect (at 86.36 88.9))
@@
     (stroke (width 0) (type default) (color 0 0 0 0))
   )
+  (wire (pts (xy 96.52 83.82) (xy 86.36 83.82))
+    (stroke (width 0) (type default) (color 0 0 0 0))
+  )
   (wire (pts (xy 153.67 175.26) (xy 149.86 175.26))
     (stroke (width 0) (type default) (color 0 0 0 0))
@@
     (stroke (width 0) (type default) (color 0 0 0 0))
   )
+  (wire (pts (xy 166.37 74.93) (xy 166.37 76.2))
+    (stroke (width 0) (type default) (color 0 0 0 0))
+  )
   (wire (pts (xy 259.08 121.92) (xy 266.7 121.92))
     (stroke (width 0) (type default) (color 0 0 0 0))
@@
     (stroke (width 0) (type default) (color 0 0 0 0))
   )
+  (wire (pts (xy 153.67 86.36) (xy 166.37 86.36))
+    (stroke (width 0) (type default) (color 0 0 0 0))
+  )
   (wire (pts (xy 55.88 124.46) (xy 55.88 125.73))
     (stroke (width 0) (type default) (color 0 0 0 0))
@@
     (stroke (width 0) (type default) (color 0 0 0 0))
   )
+  (wire (pts (xy 166.37 86.36) (xy 166.37 88.9))
+    (stroke (width 0) (type default) (color 0 0 0 0))
+  )
   (wire (pts (xy 246.38 46.99) (xy 259.08 46.99))
     (stroke (width 0) (type default) (color 0 0 0 0))
@@
     (stroke (width 0) (type default) (color 0 0 0 0))
   )
+  (wire (pts (xy 166.37 99.06) (xy 166.37 101.6))
+    (stroke (width 0) (type default) (color 0 0 0 0))
+  )
   (wire (pts (xy 130.81 99.06) (xy 130.81 104.14))
     (stroke (width 0) (type default) (color 0 0 0 0))
@@
     (stroke (width 0) (type default) (color 0 0 0 0))
   )
+  (wire (pts (xy 166.37 86.36) (xy 166.37 83.82))
+    (stroke (width 0) (type default) (color 0 0 0 0))
+  )
   (wire (pts (xy 142.24 69.85) (xy 151.13 69.85))
     (stroke (width 0) (type default) (color 0 0 0 0))
@@
     (effects (font (size 1.27 1.27)) (justify right bottom))
   )
+  (label "SHUTDOWN" (at 96.52 83.82 180)
+    (effects (font (size 1.27 1.27)) (justify right bottom))
+  )
   (label "XBEE_UART_TX" (at 17.78 148.59 0)
     (effects (font (size 1.27 1.27)) (justify left bottom))
   )
+  (label "SHUTDOWN" (at 153.67 86.36 0)
+    (effects (font (size 1.27 1.27)) (justify left bottom))
+  )
   (label "SDA" (at 266.7 119.38 180)
     (effects (font (size 1.27 1.27)) (justify right bottom))
@@
     (pin "1")
   )
+  (symbol (lib_id "power:+3V3") (at 166.37 74.93 0) (unit 1)
+    (in_bom yes) (on_board yes) (fields_autoplaced)
+    (property "Reference" "#PWR0137" (id 0) (at 166.37 78.74 0)
+      (effects (font (size 1.27 1.27)) hide)
+    )
+    (property "Value" "+3V3" (id 1) (at 166.37 69.85 0))
+    (property "Footprint" "" (id 2) (at 166.37 74.93 0)
+      (effects (font (size 1.27 1.27)) hide)
+    )
+    (property "Datasheet" "" (id 3) (at 166.37 74.93 0)
+      (effects (font (size 1.27 1.27)) hide)
+    )
+    (pin "1")
+  )
   (symbol (lib_id "power:+5V") (at 130.81 99.06 0) (unit 1)
     (in_bom yes) (on_board yes) (fields_autoplaced)
@@
     (pin "1")
   )
+  (symbol (lib_id "Switch:SW_SPST") (at 166.37 93.98 90) (mirror x) (unit 1)
+    (in_bom yes) (on_board yes) (fields_autoplaced)
+    (property "Reference" "SW1" (id 0) (at 167.64 92.7099 90)
+      (effects (font (size 1.27 1.27)) (justify right))
+    )
+    (property "Value" "SHUTDOWN" (id 1) (at 167.64 95.2499 90)
+      (effects (font (size 1.27 1.27)) (justify right))
+    )
+    (property "Footprint" "Connector_PinHeader_2.54mm:PinHeader_1x02_P2.54mm_Horizontal" (id 2) (at 166.37 93.98 0)
+      (effects (font (size 1.27 1.27)) hide)
+    )
+    (property "Datasheet" "~" (id 3) (at 166.37 93.98 0)
+      (effects (font (size 1.27 1.27)) hide)
+    )
+    (pin "1")
+    (pin "2")
+  )
   (symbol (lib_id "custom_symbols:XBee_THT") (at 63.5 168.91 0) (unit 1)
     (in_bom yes) (on_board yes) (fields_autoplaced)
@@
     (pin "2")
   )
+  (symbol (lib_id "Device:R") (at 166.37 80.01 180) (unit 1)
+    (in_bom yes) (on_board yes) (fields_autoplaced)
+    (property "Reference" "R1" (id 0) (at 163.83 78.7399 0)
+      (effects (font (size 1.27 1.27)) (justify left))
+    )
+    (property "Value" "10k" (id 1) (at 163.83 81.2799 0)
+      (effects (font (size 1.27 1.27)) (justify left))
+    )
+    (property "Footprint" "Resistor_SMD:R_0603_1608Metric" (id 2) (at 168.148 80.01 90)
+      (effects (font (size 1.27 1.27)) hide)
+    )
+    (property "Datasheet" "~" (id 3) (at 166.37 80.01 0)
+      (effects (font (size 1.27 1.27)) hide)
+    )
+    (pin "1")
+    (pin "2")
+  )
+  (symbol (lib_id "power:GND") (at 166.37 101.6 0) (unit 1)
+    (in_bom yes) (on_board yes) (fields_autoplaced)
+    (property "Reference" "#PWR0138" (id 0) (at 166.37 107.95 0)
+      (effects (font (size 1.27 1.27)) hide)
+    )
+    (property "Value" "GND" (id 1) (at 166.37 106.68 0))
+    (property "Footprint" "" (id 2) (at 166.37 101.6 0)
+      (effects (font (size 1.27 1.27)) hide)
+    )
+    (property "Datasheet" "" (id 3) (at 166.37 101.6 0)
+      (effects (font (size 1.27 1.27)) hide)
+    )
+    (pin "1")
+  )
   (symbol (lib_id "Device:C_Small") (at 114.3 54.61 0) (unit 1)
     (in_bom yes) (on_board yes) (fields_autoplaced)
@@
       (reference "#PWR0136") (unit 1) (value "+3V3") (footprint "")
     )
+    (path "/0b389c6b-fa33-4abf-8603-f8c0245617d0"
+      (reference "#PWR0137") (unit 1) (value "+3V3") (footprint "")
+    )
+    (path "/ce668996-e554-4203-9697-5d27959007c1"
+      (reference "#PWR0138") (unit 1) (value "GND") (footprint "")
+    )
     (path "/dce5d536-e66b-40aa-9add-0f38dedf7b75"
       (reference "BZ1") (unit 1) (value "Buzzer") (footprint "custom-footprints:CPI-1375-80T")
@@
       (reference "Q1") (unit 2) (value "AO4838") (footprint "Package_SO:SOIC-8_3.9x4.9mm_P1.27mm")
     )
+    (path "/ccb2cfb8-7cb4-43f3-9d28-b55ed24ad453"
+      (reference "R1") (unit 1) (value "10k") (footprint "Resistor_SMD:R_0603_1608Metric")
+    )
     (path "/e3dd2361-8a26-4d67-8fa2-04aedf170f2c/13c198e3-2d63-467b-8892-241e6450945b"
       (reference "R3") (unit 1) (value "100k") (footprint "Resistor_SMD:R_0603_1608Metric")
@@
       (reference "S7") (unit 1) (value "Conn_01x03_Male") (footprint "Connector_PinHeader_2.54mm:PinHeader_1x03_P2.54mm_Vertical")
     )
+    (path "/3cbec5a9-3d9e-4d6e-b914-0c15fc69d431"
+      (reference "SW1") (unit 1) (value "SHUTDOWN") (footprint "Connector_PinHeader_2.54mm:PinHeader_1x02_P2.54mm_Horizontal")
+    )
     (path "/bcffcd1c-cbf8-4b45-8e7d-e9d4037cabb3"
