File: Motherboard/motherboard_2022_2023/pyro_channel_pair.kicad_sch (KiCad schematic)
At the start: 11 parts, among them J11 Conn_01x02, J12 Conn_01x02, Q1 AO4838

Commit message: Added SDA/SCL & Document Titles
Parts:
- renumbered R8 to R10, R9 to R11, R10 to R12, R5 to R7, R6 to R8, R7 to R9
Other:
- company: (none) -> Rose-Hulman Institute of Technology
- title: (none) -> High-Current Channel Output Control
Changed lines of the file:
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@@
 (kicad_sch (version 20211123) (generator eeschema)
   (paper "A4")
+  (title_block
+    (title "High-Current Channel Output Control")
+    (date "2022-10-23")
+    (rev "1.0")
+    (company "Rose-Hulman Institute of Technology")
+    (comment 1 "Author: Evelyn Gordon")
+    (comment 2 "For Rose Rocketry")
+  )
   (junction (at 64.77 82.55) (diameter 0) (color 0 0 0 0)
   )
@@
   (symbol (lib_id "Device:R") (at 36.83 50.8 0) (unit 1)
     (in_bom yes) (on_board yes) (fields_autoplaced)
-    (property "Reference" "R5" (id 0) (at 39.37 49.5299 0)
+    (property "Reference" "R7" (id 0) (at 39.37 49.5299 0)
       (effects (font (size 1.27 1.27)) (justify left))
     )
@@
   (symbol (lib_id "power:GND") (at 48.26 125.73 0) (unit 1)
     (in_bom yes) (on_board yes) (fields_autoplaced)
-    (property "Reference" "#PWR0116" (id 0) (at 48.26 132.08 0)
+    (property "Reference" "#PWR023" (id 0) (at 48.26 132.08 0)
       (effects (font (size 1.27 1.27)) hide)
     )
@@
   (symbol (lib_id "Device:R") (at 64.77 60.96 0) (unit 1)
     (in_bom yes) (on_board yes) (fields_autoplaced)
-    (property "Reference" "R8" (id 0) (at 67.31 59.6899 0)
+    (property "Reference" "R10" (id 0) (at 67.31 59.6899 0)
       (effects (font (size 1.27 1.27)) (justify left))
     )
@@
   (symbol (lib_id "Device:R") (at 64.77 118.11 0) (unit 1)
     (in_bom yes) (on_board yes) (fields_autoplaced)
-    (property "Reference" "R10" (id 0) (at 67.31 116.8399 0)
+    (property "Reference" "R12" (id 0) (at 67.31 116.8399 0)
       (effects (font (size 1.27 1.27)) (justify left))
     )
@@
   (symbol (lib_id "Device:R") (at 36.83 107.95 0) (unit 1)
     (in_bom yes) (on_board yes) (fields_autoplaced)
-    (property "Reference" "R6" (id 0) (at 39.37 106.6799 0)
+    (property "Reference" "R8" (id 0) (at 39.37 106.6799 0)
       (effects (font (size 1.27 1.27)) (justify left))
     )
@@
   (symbol (lib_id "power:GND") (at 48.26 68.58 0) (unit 1)
     (in_bom yes) (on_board yes) (fields_autoplaced)
-    (property "Reference" "#PWR0115" (id 0) (at 48.26 74.93 0)
+    (property "Reference" "#PWR022" (id 0) (at 48.26 74.93 0)
       (effects (font (size 1.27 1.27)) hide)
     )
@@
   (symbol (lib_id "Device:R") (at 64.77 105.41 0) (unit 1)
     (in_bom yes) (on_board yes) (fields_autoplaced)
-    (property "Reference" "R9" (id 0) (at 67.31 104.1399 0)
+    (property "Reference" "R11" (id 0) (at 67.31 104.1399 0)
       (effects (font (size 1.27 1.27)) (justify left))
     )
@@
   (symbol (lib_id "Device:R") (at 64.77 48.26 0) (unit 1)
     (in_bom yes) (on_board yes) (fields_autoplaced)
-    (property "Reference" "R7" (id 0) (at 67.31 46.9899 0)
-      (effects (font (size 1.27 1.27)) (justify left))
-    )
+    (property "Reference" "R9" (id 0) (at 67.31 46.9899 0)
+      (effects (font (size 1.27 1.27)) (justify left))
+    )

Commit message: Update 3d models
Parts:
- J11, J12: footprint TerminalBlock:TerminalBlock_bornier-2_P5.08mm -> TerminalBlock_Phoenix:TerminalBlock_Phoenix_PT-1,5-2-5.0-H_1x02_P5.00mm_Horizontal
Changed lines of the file:
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@@
       (effects (font (size 1.27 1.27)) (justify left))
     )
-    (property "Footprint" "TerminalBlock:TerminalBlock_bornier-2_P5.08mm" (id 2) (at 80.01 22.86 0)
+    (property "Footprint" "TerminalBlock_Phoenix:TerminalBlock_Phoenix_PT-1,5-2-5.0-H_1x02_P5.00mm_Horizontal" (id 2) (at 80.01 22.86 0)
       (effects (font (size 1.27 1.27)) hide)
     )
@@
       (effects (font (size 1.27 1.27)) (justify left))
     )
-    (property "Footprint" "TerminalBlock:TerminalBlock_bornier-2_P5.08mm" (id 2) (at 80.01 80.01 0)
+    (property "Footprint" "TerminalBlock_Phoenix:TerminalBlock_Phoenix_PT-1,5-2-5.0-H_1x02_P5.00mm_Horizontal" (id 2) (at 80.01 80.01 0)
       (effects (font (size 1.27 1.27)) hide)
     )

Commit message: Added Resistors to MOSFET at Ben's Request
Parts:
- added R14, R15: 220, Resistor_SMD:R_0603_1608Metric, symbol Device:R
- R7, R8: value 100k -> 10k
Connections:
- net PYRO_A: now also R14.1; no longer Q1.2 (G)
- net PYRO_B: now also R15.1; no longer Q1.4 (G)
- new net: Q1.4 (G), R15.2
- new net: Q1.2 (G), R14.2
Other:
- moved on the sheet: R7, R8
Changed lines of the file:
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@@
   (junction (at 50.8 25.4) (diameter 0) (color 0 0 0 0)
   )
+  (junction (at 29.21 92.71) (diameter 0) (color 0 0 0 0)
+  )
   (junction (at 48.26 123.19) (diameter 0) (color 0 0 0 0)
   )
-  (junction (at 36.83 92.71) (diameter 0) (color 0 0 0 0)
-  )
   (junction (at 64.77 111.76) (diameter 0) (color 0 0 0 0)
   )
-  (junction (at 36.83 35.56) (diameter 0) (color 0 0 0 0)
+  (junction (at 31.75 35.56) (diameter 0) (color 0 0 0 0)
   )
   (junction (at 64.77 54.61) (diameter 0) (color 0 0 0 0)
@@
     (stroke (width 0) (type default) (color 0 0 0 0))
   )
-  (wire (pts (xy 36.83 35.56) (xy 36.83 46.99))
+  (wire (pts (xy 31.75 35.56) (xy 31.75 46.99))
     (stroke (width 0) (type default) (color 0 0 0 0))
   )
@@
     (stroke (width 0) (type default) (color 0 0 0 0))
   )
-  (wire (pts (xy 36.83 35.56) (xy 40.64 35.56))
+  (wire (pts (xy 31.75 35.56) (xy 33.02 35.56))
     (stroke (width 0) (type default) (color 0 0 0 0))
   )
@@
     (stroke (width 0) (type default) (color 0 0 0 0))
   )
-  (wire (pts (xy 36.83 123.19) (xy 48.26 123.19))
+  (wire (pts (xy 29.21 123.19) (xy 48.26 123.19))
+    (stroke (width 0) (type default) (color 0 0 0 0))
+  )
+  (wire (pts (xy 29.21 35.56) (xy 31.75 35.56))
     (stroke (width 0) (type default) (color 0 0 0 0))
   )
@@
     (stroke (width 0) (type default) (color 0 0 0 0))
   )
-  (wire (pts (xy 36.83 111.76) (xy 36.83 123.19))
+  (wire (pts (xy 29.21 111.76) (xy 29.21 123.19))
     (stroke (width 0) (type default) (color 0 0 0 0))
   )
@@
     (stroke (width 0) (type default) (color 0 0 0 0))
   )
+  (wire (pts (xy 39.37 35.56) (xy 40.64 35.56))
+    (stroke (width 0) (type default) (color 0 0 0 0))
+  )
+  (wire (pts (xy 29.21 92.71) (xy 31.75 92.71))
+    (stroke (width 0) (type default) (color 0 0 0 0))
+  )
   (wire (pts (xy 50.8 25.4) (xy 64.77 25.4))
     (stroke (width 0) (type default) (color 0 0 0 0))
@@
     (stroke (width 0) (type default) (color 0 0 0 0))
   )
-  (wire (pts (xy 33.02 92.71) (xy 36.83 92.71))
-    (stroke (width 0) (type default) (color 0 0 0 0))
-  )
-  (wire (pts (xy 36.83 54.61) (xy 36.83 66.04))
-    (stroke (width 0) (type default) (color 0 0 0 0))
-  )
-  (wire (pts (xy 36.83 92.71) (xy 36.83 104.14))
-    (stroke (width 0) (type default) (color 0 0 0 0))
-  )
-  (wire (pts (xy 36.83 66.04) (xy 48.26 66.04))
+  (wire (pts (xy 31.75 54.61) (xy 31.75 66.04))
+    (stroke (width 0) (type default) (color 0 0 0 0))
+  )
+  (wire (pts (xy 29.21 92.71) (xy 29.21 104.14))
+    (stroke (width 0) (type default) (color 0 0 0 0))
+  )
+  (wire (pts (xy 26.67 92.71) (xy 29.21 92.71))
+    (stroke (width 0) (type default) (color 0 0 0 0))
+  )
+  (wire (pts (xy 31.75 66.04) (xy 48.26 66.04))
     (stroke (width 0) (type default) (color 0 0 0 0))
   )
@@
     (stroke (width 0) (type default) (color 0 0 0 0))
   )
-  (wire (pts (xy 36.83 92.71) (xy 40.64 92.71))
+  (wire (pts (xy 39.37 92.71) (xy 40.64 92.71))
     (stroke (width 0) (type default) (color 0 0 0 0))
   )
@@
     (stroke (width 0) (type default) (color 0 0 0 0))
   )
-  (wire (pts (xy 33.02 35.56) (xy 36.83 35.56))
-    (stroke (width 0) (type default) (color 0 0 0 0))
-  )
   (wire (pts (xy 64.77 25.4) (xy 64.77 31.75))
     (stroke (width 0) (type default) (color 0 0 0 0))
@@
     (stroke (width 0) (type default) (color 0 0 0 0))
   )
-  (hierarchical_label "PYRO_A" (shape input) (at 33.02 35.56 180)
+  (hierarchical_label "PYRO_A" (shape input) (at 29.21 35.56 180)
     (effects (font (size 1.27 1.27)) (justify right))
   )
@@
     (effects (font (size 1.27 1.27)) (justify right))
   )
-  (hierarchical_label "PYRO_B" (shape input) (at 33.02 92.71 180)
+  (hierarchical_label "PYRO_B" (shape input) (at 26.67 92.71 180)
     (effects (font (size 1.27 1.27)) (justify right))
   )
@@
     (effects (font (size 1.27 1.27)) (justify right))
   )
-  (symbol (lib_id "Device:R") (at 36.83 50.8 0) (unit 1)
-    (in_bom yes) (on_board yes) (fields_autoplaced)
-    (property "Reference" "R7" (id 0) (at 39.37 49.5299 0)
-      (effects (font (size 1.27 1.27)) (justify left))
-    )
-    (property "Value" "100k" (id 1) (at 39.37 52.0699 0)
-      (effects (font (size 1.27 1.27)) (justify left))
-    )
-    (property "Footprint" "Resistor_SMD:R_0603_1608Metric" (id 2) (at 35.052 50.8 90)
-      (effects (font (size 1.27 1.27)) hide)
-    )
-    (property "Datasheet" "~" (id 3) (at 36.83 50.8 0)
+  (symbol (lib_id "Device:R") (at 31.75 50.8 0) (unit 1)
+    (in_bom yes) (on_board yes) (fields_autoplaced)
+    (property "Reference" "R7" (id 0) (at 34.29 49.5299 0)
+      (effects (font (size 1.27 1.27)) (justify left))
+    )
+    (property "Value" "10k" (id 1) (at 34.29 52.0699 0)
+      (effects (font (size 1.27 1.27)) (justify left))
+    )
+    (property "Footprint" "Resistor_SMD:R_0603_1608Metric" (id 2) (at 29.972 50.8 90)
+      (effects (font (size 1.27 1.27)) hide)
+    )
+    (property "Datasheet" "~" (id 3) (at 31.75 50.8 0)
       (effects (font (size 1.27 1.27)) hide)
     )
@@
     (pin "2")
   )
-  (symbol (lib_id "Device:R") (at 36.83 107.95 0) (unit 1)
-    (in_bom yes) (on_board yes) (fields_autoplaced)
-    (property "Reference" "R8" (id 0) (at 39.37 106.6799 0)
-      (effects (font (size 1.27 1.27)) (justify left))
-    )
-    (property "Value" "100k" (id 1) (at 39.37 109.2199 0)
-      (effects (font (size 1.27 1.27)) (justify left))
-    )
-    (property "Footprint" "Resistor_SMD:R_0603_1608Metric" (id 2) (at 35.052 107.95 90)
-      (effects (font (size 1.27 1.27)) hide)
-    )
-    (property "Datasheet" "~" (id 3) (at 36.83 107.95 0)
-      (effects (font (size 1.27 1.27)) hide)
-    )
+  (symbol (lib_id "Device:R") (at 35.56 92.71 90) (unit 1)
+    (in_bom yes) (on_board yes) (fields_autoplaced)
+    (property "Reference" "R15" (id 0) (at 35.56 86.36 90))
+    (property "Value" "220" (id 1) (at 35.56 88.9 90))
+    (property "Footprint" "Resistor_SMD:R_0603_1608Metric" (id 2) (at 35.56 94.488 90)
+      (effects (font (size 1.27 1.27)) hide)
+    )
+    (property "Datasheet" "~" (id 3) (at 35.56 92.71 0)
+      (effects (font (size 1.27 1.27)) hide)
+    )
+    (pin "1")
+    (pin "2")
+  )
+  (symbol (lib_id "Device:R") (at 35.56 35.56 90) (unit 1)
+    (in_bom yes) (on_board yes) (fields_autoplaced)
+    (property "Reference" "R14" (id 0) (at 35.56 29.21 90))
+    (property "Value" "220" (id 1) (at 35.56 31.75 90))
+    (property "Footprint" "Resistor_SMD:R_0603_1608Metric" (id 2) (at 35.56 37.338 90)
+      (effects (font (size 1.27 1.27)) hide)
+    )
+    (property "Datasheet" "~" (id 3) (at 35.56 35.56 0)
+      (effects (font (size 1.27 1.27)) hide)
+    )
+    (pin "1")
+    (pin "2")
+  )
+  (symbol (lib_id "Device:R") (at 29.21 107.95 0) (unit 1)
+    (in_bom yes) (on_board yes) (fields_autoplaced)
+    (property "Reference" "R8" (id 0) (at 31.75 106.6799 0)
+      (effects (font (size 1.27 1.27)) (justify left))
+    )
+    (property "Value" "10k" (id 1) (at 31.75 109.2199 0)
+      (effects (font (size 1.27 1.27)) (justify left))
+    )
+    (property "Footprint" "Resistor_SMD:R_0603_1608Metric" (id 2) (at 27.432 107.95 90)
+      (effects (font (size 1.27 1.27)) hide)
+    )
+    (property "Datasheet" "~" (id 3) (at 29.21 107.95 0)
+      (effects (font (size 1.27 1.27)) hide)
+    )
