File: Motherboard/motherboard_2022_2023/pyro_channel_pair.kicad_sch (KiCad schematic)
At the start: 13 parts, among them J11 Conn_01x02, J12 Conn_01x02, Q1 AO4838

Commit message: Route rest of PCB, passes almost all meaningful DRC
Other:
- moved on the sheet: R7
Changed lines of the file:
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@@
   (junction (at 64.77 111.76) (diameter 0) (color 0 0 0 0)
   )
-  (junction (at 31.75 35.56) (diameter 0) (color 0 0 0 0)
-  )
   (junction (at 64.77 54.61) (diameter 0) (color 0 0 0 0)
   )
   (junction (at 64.77 25.4) (diameter 0) (color 0 0 0 0)
   )
+  (junction (at 29.21 35.56) (diameter 0) (color 0 0 0 0)
+  )
   (junction (at 48.26 66.04) (diameter 0) (color 0 0 0 0)
   )
@@
     (stroke (width 0) (type default) (color 0 0 0 0))
   )
-  (wire (pts (xy 31.75 35.56) (xy 31.75 46.99))
+  (wire (pts (xy 29.21 35.56) (xy 29.21 46.99))
     (stroke (width 0) (type default) (color 0 0 0 0))
   )
@@
     (stroke (width 0) (type default) (color 0 0 0 0))
   )
-  (wire (pts (xy 31.75 35.56) (xy 33.02 35.56))
-    (stroke (width 0) (type default) (color 0 0 0 0))
-  )
   (wire (pts (xy 39.37 80.01) (xy 74.93 80.01))
     (stroke (width 0) (type default) (color 0 0 0 0))
@@
     (stroke (width 0) (type default) (color 0 0 0 0))
   )
+  (wire (pts (xy 26.67 35.56) (xy 29.21 35.56))
+    (stroke (width 0) (type default) (color 0 0 0 0))
+  )
+  (wire (pts (xy 48.26 97.79) (xy 48.26 123.19))
+    (stroke (width 0) (type default) (color 0 0 0 0))
+  )
+  (wire (pts (xy 29.21 111.76) (xy 29.21 123.19))
+    (stroke (width 0) (type default) (color 0 0 0 0))
+  )
+  (wire (pts (xy 64.77 109.22) (xy 64.77 111.76))
+    (stroke (width 0) (type default) (color 0 0 0 0))
+  )
+  (wire (pts (xy 39.37 35.56) (xy 40.64 35.56))
+    (stroke (width 0) (type default) (color 0 0 0 0))
+  )
+  (wire (pts (xy 29.21 92.71) (xy 31.75 92.71))
+    (stroke (width 0) (type default) (color 0 0 0 0))
+  )
+  (wire (pts (xy 50.8 25.4) (xy 64.77 25.4))
+    (stroke (width 0) (type default) (color 0 0 0 0))
+  )
+  (wire (pts (xy 48.26 123.19) (xy 64.77 123.19))
+    (stroke (width 0) (type default) (color 0 0 0 0))
+  )
   (wire (pts (xy 29.21 35.56) (xy 31.75 35.56))
     (stroke (width 0) (type default) (color 0 0 0 0))
   )
-  (wire (pts (xy 48.26 97.79) (xy 48.26 123.19))
-    (stroke (width 0) (type default) (color 0 0 0 0))
-  )
-  (wire (pts (xy 29.21 111.76) (xy 29.21 123.19))
-    (stroke (width 0) (type default) (color 0 0 0 0))
-  )
-  (wire (pts (xy 64.77 109.22) (xy 64.77 111.76))
-    (stroke (width 0) (type default) (color 0 0 0 0))
-  )
-  (wire (pts (xy 39.37 35.56) (xy 40.64 35.56))
-    (stroke (width 0) (type default) (color 0 0 0 0))
-  )
-  (wire (pts (xy 29.21 92.71) (xy 31.75 92.71))
-    (stroke (width 0) (type default) (color 0 0 0 0))
-  )
-  (wire (pts (xy 50.8 25.4) (xy 64.77 25.4))
-    (stroke (width 0) (type default) (color 0 0 0 0))
-  )
-  (wire (pts (xy 48.26 123.19) (xy 64.77 123.19))
-    (stroke (width 0) (type default) (color 0 0 0 0))
-  )
   (wire (pts (xy 64.77 66.04) (xy 64.77 64.77))
     (stroke (width 0) (type default) (color 0 0 0 0))
@@
     (stroke (width 0) (type default) (color 0 0 0 0))
   )
-  (wire (pts (xy 31.75 54.61) (xy 31.75 66.04))
+  (wire (pts (xy 29.21 54.61) (xy 29.21 66.04))
     (stroke (width 0) (type default) (color 0 0 0 0))
   )
@@
     (stroke (width 0) (type default) (color 0 0 0 0))
   )
-  (wire (pts (xy 31.75 66.04) (xy 48.26 66.04))
+  (wire (pts (xy 29.21 66.04) (xy 48.26 66.04))
     (stroke (width 0) (type default) (color 0 0 0 0))
   )
@@
     (stroke (width 0) (type default) (color 0 0 0 0))
   )
-  (hierarchical_label "PYRO_A" (shape input) (at 29.21 35.56 180)
+  (hierarchical_label "PYRO_A" (shape input) (at 26.67 35.56 180)
     (effects (font (size 1.27 1.27)) (justify right))
   )
@@
     (effects (font (size 1.27 1.27)) (justify right))
   )
-  (symbol (lib_id "Device:R") (at 31.75 50.8 0) (unit 1)
-    (in_bom yes) (on_board yes) (fields_autoplaced)
-    (property "Reference" "R7" (id 0) (at 34.29 49.5299 0)
-      (effects (font (size 1.27 1.27)) (justify left))
-    )
-    (property "Value" "10k" (id 1) (at 34.29 52.0699 0)
-      (effects (font (size 1.27 1.27)) (justify left))
-    )
-    (property "Footprint" "Resistor_SMD:R_0603_1608Metric" (id 2) (at 29.972 50.8 90)
-      (effects (font (size 1.27 1.27)) hide)
-    )
-    (property "Datasheet" "~" (id 3) (at 31.75 50.8 0)
+  (symbol (lib_id "Device:R") (at 29.21 50.8 0) (unit 1)
+    (in_bom yes) (on_board yes) (fields_autoplaced)
+    (property "Reference" "R7" (id 0) (at 31.75 49.5299 0)
+      (effects (font (size 1.27 1.27)) (justify left))
+    )
+    (property "Value" "10k" (id 1) (at 31.75 52.0699 0)
+      (effects (font (size 1.27 1.27)) (justify left))
+    )
+    (property "Footprint" "Resistor_SMD:R_0603_1608Metric" (id 2) (at 27.432 50.8 90)
+      (effects (font (size 1.27 1.27)) hide)
+    )
+    (property "Datasheet" "~" (id 3) (at 29.21 50.8 0)
       (effects (font (size 1.27 1.27)) hide)
     )
@@
       (effects (font (size 1.27 1.27)) hide)
     )
+    (pin "1")
+    (pin "2")
+    (pin "7")
+    (pin "8")
     (pin "3")
     (pin "4")
@@
     (pin "7")
     (pin "8")
+    (pin "3")
+    (pin "4")
+    (pin "5")
+    (pin "6")
   )
   (symbol (lib_id "Connector_Generic:Conn_01x02") (at 80.01 22.86 0) (unit 1)

Commit message: Add HDMI adaptor
Parts:
- added D1: 3v3, symbol Device:D_Zener
- R11, R9: value 200k -> 100k
Connections:
- net GND: now also D1.2 (A)
- net PYRO_A_SENSE: now also D1.1 (K)
Changed lines of the file:
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@@
   (junction (at 48.26 123.19) (diameter 0) (color 0 0 0 0)
   )
+  (junction (at 54.61 66.04) (diameter 0) (color 0 0 0 0)
+  )
+  (junction (at 64.77 54.61) (diameter 0) (color 0 0 0 0)
+  )
+  (junction (at 64.77 25.4) (diameter 0) (color 0 0 0 0)
+  )
+  (junction (at 54.61 123.19) (diameter 0) (color 0 0 0 0)
+  )
+  (junction (at 29.21 35.56) (diameter 0) (color 0 0 0 0)
+  )
+  (junction (at 48.26 66.04) (diameter 0) (color 0 0 0 0)
+  )
   (junction (at 64.77 111.76) (diameter 0) (color 0 0 0 0)
   )
-  (junction (at 64.77 54.61) (diameter 0) (color 0 0 0 0)
-  )
-  (junction (at 64.77 25.4) (diameter 0) (color 0 0 0 0)
-  )
-  (junction (at 29.21 35.56) (diameter 0) (color 0 0 0 0)
-  )
-  (junction (at 48.26 66.04) (diameter 0) (color 0 0 0 0)
-  )
   (wire (pts (xy 64.77 96.52) (xy 64.77 101.6))
     (stroke (width 0) (type default) (color 0 0 0 0))
@@
     (stroke (width 0) (type default) (color 0 0 0 0))
   )
+  (wire (pts (xy 54.61 114.3) (xy 54.61 111.76))
+    (stroke (width 0) (type default) (color 0 0 0 0))
+  )
   (wire (pts (xy 64.77 82.55) (xy 74.93 82.55))
     (stroke (width 0) (type default) (color 0 0 0 0))
@@
     (stroke (width 0) (type default) (color 0 0 0 0))
   )
+  (wire (pts (xy 54.61 57.15) (xy 54.61 54.61))
+    (stroke (width 0) (type default) (color 0 0 0 0))
+  )
   (wire (pts (xy 39.37 80.01) (xy 74.93 80.01))
     (stroke (width 0) (type default) (color 0 0 0 0))
   )
-  (wire (pts (xy 48.26 66.04) (xy 64.77 66.04))
+  (wire (pts (xy 48.26 66.04) (xy 54.61 66.04))
     (stroke (width 0) (type default) (color 0 0 0 0))
   )
@@
     (stroke (width 0) (type default) (color 0 0 0 0))
   )
+  (wire (pts (xy 54.61 66.04) (xy 64.77 66.04))
+    (stroke (width 0) (type default) (color 0 0 0 0))
+  )
   (wire (pts (xy 48.26 25.4) (xy 48.26 30.48))
     (stroke (width 0) (type default) (color 0 0 0 0))
@@
     (stroke (width 0) (type default) (color 0 0 0 0))
   )
+  (wire (pts (xy 64.77 111.76) (xy 64.77 114.3))
+    (stroke (width 0) (type default) (color 0 0 0 0))
+  )
   (wire (pts (xy 64.77 109.22) (xy 64.77 111.76))
     (stroke (width 0) (type default) (color 0 0 0 0))
@@
     (stroke (width 0) (type default) (color 0 0 0 0))
   )
-  (wire (pts (xy 48.26 123.19) (xy 64.77 123.19))
+  (wire (pts (xy 48.26 123.19) (xy 54.61 123.19))
     (stroke (width 0) (type default) (color 0 0 0 0))
   )
@@
     (stroke (width 0) (type default) (color 0 0 0 0))
   )
+  (wire (pts (xy 54.61 123.19) (xy 64.77 123.19))
+    (stroke (width 0) (type default) (color 0 0 0 0))
+  )
   (wire (pts (xy 64.77 123.19) (xy 64.77 121.92))
     (stroke (width 0) (type default) (color 0 0 0 0))
   )
+  (wire (pts (xy 64.77 111.76) (xy 68.58 111.76))
+    (stroke (width 0) (type default) (color 0 0 0 0))
+  )
   (wire (pts (xy 50.8 82.55) (xy 48.26 82.55))
     (stroke (width 0) (type default) (color 0 0 0 0))
   )
+  (wire (pts (xy 54.61 64.77) (xy 54.61 66.04))
+    (stroke (width 0) (type default) (color 0 0 0 0))
+  )
   (wire (pts (xy 29.21 54.61) (xy 29.21 66.04))
     (stroke (width 0) (type default) (color 0 0 0 0))
@@
     (stroke (width 0) (type default) (color 0 0 0 0))
   )
+  (wire (pts (xy 54.61 54.61) (xy 64.77 54.61))
+    (stroke (width 0) (type default) (color 0 0 0 0))
+  )
   (wire (pts (xy 26.67 92.71) (xy 29.21 92.71))
     (stroke (width 0) (type default) (color 0 0 0 0))
@@
     (stroke (width 0) (type default) (color 0 0 0 0))
   )
+  (wire (pts (xy 54.61 121.92) (xy 54.61 123.19))
+    (stroke (width 0) (type default) (color 0 0 0 0))
+  )
   (wire (pts (xy 39.37 92.71) (xy 40.64 92.71))
     (stroke (width 0) (type default) (color 0 0 0 0))
@@
     (stroke (width 0) (type default) (color 0 0 0 0))
   )
-  (wire (pts (xy 64.77 111.76) (xy 64.77 114.3))
-    (stroke (width 0) (type default) (color 0 0 0 0))
-  )
   (wire (pts (xy 48.26 40.64) (xy 48.26 66.04))
     (stroke (width 0) (type default) (color 0 0 0 0))
@@
     (stroke (width 0) (type default) (color 0 0 0 0))
   )
-  (wire (pts (xy 64.77 111.76) (xy 68.58 111.76))
+  (wire (pts (xy 54.61 111.76) (xy 64.77 111.76))
     (stroke (width 0) (type default) (color 0 0 0 0))
   )
@@
       (effects (font (size 1.27 1.27)) (justify left))
     )
-    (property "Value" "200k" (id 1) (at 67.31 106.6799 0)
+    (property "Value" "100k" (id 1) (at 67.31 106.6799 0)
       (effects (font (size 1.27 1.27)) (justify left))
     )
@@
       (effects (font (size 1.27 1.27)) (justify left))
     )
-    (property "Value" "200k" (id 1) (at 67.31 49.5299 0)
+    (property "Value" "100k" (id 1) (at 67.31 49.5299 0)
       (effects (font (size 1.27 1.27)) (justify left))
     )
@@
       (effects (font (size 1.27 1.27)) hide)
     )
+    (pin "1")
+    (pin "2")
+  )
+  (symbol (lib_id "Device:D_Zener") (at 54.61 60.96 270) (unit 1)
+    (in_bom yes) (on_board yes) (fields_autoplaced)
+    (property "Reference" "D1" (id 0) (at 57.15 59.6899 90)
+      (effects (font (size 1.27 1.27)) (justify left))
+    )
+    (property "Value" "3v3" (id 1) (at 57.15 62.2299 90)
+      (effects (font (size 1.27 1.27)) (justify left))
+    )
+    (property "Footprint" "" (id 2) (at 54.61 60.96 0)
+      (effects (font (size 1.27 1.27)) hide)
+    )
+    (property "Datasheet" "~" (id 3) (at 54.61 60.96 0)
+      (effects (font (size 1.27 1.27)) hide)
+    )

Commit message: Add mousebite
Parts:
- added D2: 3v3, Diode_THT:D_DO-41_SOD81_P2.54mm_Vertical_AnodeUp, symbol Device:D_Zener
- D1: footprint (none) -> Diode_THT:D_DO-41_SOD81_P2.54mm_Vertical_AnodeUp
Connections:
- net GND: now also D2.2 (A)
- net PYRO_B_SENSE: now also D2.1 (K)
Changed lines of the file:
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@@
     (pin "6")
+  )
+  (symbol (lib_id "Device:D_Zener") (at 54.61 118.11 270) (unit 1)
+    (in_bom yes) (on_board yes) (fields_autoplaced)
+    (property "Reference" "D2" (id 0) (at 57.15 116.8399 90)
+      (effects (font (size 1.27 1.27)) (justify left))
+    )
+    (property "Value" "3v3" (id 1) (at 57.15 119.3799 90)
+      (effects (font (size 1.27 1.27)) (justify left))
+    )
+    (property "Footprint" "Diode_THT:D_DO-41_SOD81_P2.54mm_Vertical_AnodeUp" (id 2) (at 54.61 118.11 0)
+      (effects (font (size 1.27 1.27)) hide)
+    )
+    (property "Datasheet" "~" (id 3) (at 54.61 118.11 0)
+      (effects (font (size 1.27 1.27)) hide)
+    )
+    (pin "1")
+    (pin "2")
   )
   (symbol (lib_id "Connector_Generic:Conn_01x02") (at 80.01 22.86 0) (unit 1)
@@
       (effects (font (size 1.27 1.27)) (justify left))
     )
-    (property "Footprint" "" (id 2) (at 54.61 60.96 0)
+    (property "Footprint" "Diode_THT:D_DO-41_SOD81_P2.54mm_Vertical_AnodeUp" (id 2) (at 54.61 60.96 0)
       (effects (font (size 1.27 1.27)) hide)
     )
