File: Motherboard/motherboard_2022_2023/pyro_channel_pair.kicad_sch (KiCad schematic)
At the start: 15 parts, among them J11 Conn_01x02, J12 Conn_01x02, Q1 AO4838

Commit message: Use correct footprint for screw terminals
Parts:
- removed J11, J12: Conn_01x02, TerminalBlock_Phoenix:TerminalBlock_Phoenix_PT-1,5-2-5.0-H_1x02_P5.00mm_Horizontal, symbol Connector_Generic:Conn_01x02
- added J5: Screw_Terminal_01x04, TerminalBlock_Phoenix:TerminalBlock_Phoenix_MPT-0,5-4-2.54_1x04_P2.54mm_Horizontal, symbol Connector:Screw_Terminal_01x04
Connections:
- net V_BAT: now also J5.1 (Pin_1), J5.3 (Pin_3)
- net PYRO_A_PWR: now reaches JP1.2 (B), Q1.7 (D), Q1.8 (D)
- net PYRO_A_PWR: now also J5.4 (Pin_4)
- net PYRO_B_PWR: now reaches JP2.2 (B), Q1.5 (D), Q1.6 (D)
- net PYRO_B_PWR: now also J5.2 (Pin_2)
Changed lines of the file:
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@@
+    (stroke (width 0) (type default) (color 0 0 0 0))
+  )
+  (wire (pts (xy 93.98 33.02) (xy 107.95 33.02))
     (stroke (width 0) (type default) (color 0 0 0 0))
   )
@@
     (stroke (width 0) (type default) (color 0 0 0 0))
   )
-  (wire (pts (xy 39.37 80.01) (xy 74.93 80.01))
-    (stroke (width 0) (type default) (color 0 0 0 0))
-  )
   (wire (pts (xy 48.26 66.04) (xy 54.61 66.04))
     (stroke (width 0) (type default) (color 0 0 0 0))
@@
     (stroke (width 0) (type default) (color 0 0 0 0))
   )
+  (wire (pts (xy 93.98 38.1) (xy 107.95 38.1))
+    (stroke (width 0) (type default) (color 0 0 0 0))
+  )
   (wire (pts (xy 50.8 82.55) (xy 50.8 87.63))
     (stroke (width 0) (type default) (color 0 0 0 0))
@@
   )
   (wire (pts (xy 29.21 66.04) (xy 48.26 66.04))
-    (stroke (width 0) (type default) (color 0 0 0 0))
-  )
-  (wire (pts (xy 39.37 22.86) (xy 74.93 22.86))
     (stroke (width 0) (type default) (color 0 0 0 0))
   )
@@
     )
   )
+  (label "PYRO_B_PWR" (at 93.98 38.1 0)
+    (effects (font (size 1.27 1.27)) (justify left bottom))
+  )
+  (label "PYRO_B_PWR" (at 74.93 82.55 180)
+    (effects (font (size 1.27 1.27)) (justify right bottom))
+  )
+  (label "PYRO_A_PWR" (at 93.98 33.02 0)
+    (effects (font (size 1.27 1.27)) (justify left bottom))
+  )
+  (label "PYRO_A_PWR" (at 74.93 25.4 180)
+    (effects (font (size 1.27 1.27)) (justify right bottom))
+  )
   (hierarchical_label "PYRO_A" (shape input) (at 26.67 35.56 180)
     (effects (font (size 1.27 1.27)) (justify right))
@@
     (effects (font (size 1.27 1.27)) (justify left))
   )
-  (hierarchical_label "V_BAT" (shape input) (at 39.37 22.86 180)
-    (effects (font (size 1.27 1.27)) (justify right))
-  )
   (hierarchical_label "PYRO_B" (shape input) (at 26.67 92.71 180)
     (effects (font (size 1.27 1.27)) (justify right))
   )
-  (hierarchical_label "V_BAT" (shape input) (at 39.37 80.01 180)
+  (hierarchical_label "V_BAT" (shape input) (at 107.95 35.56 180)
+    (effects (font (size 1.27 1.27)) (justify right))
+  )
+  (hierarchical_label "V_BAT" (shape input) (at 107.95 40.64 180)
     (effects (font (size 1.27 1.27)) (justify right))
   )
@@
     )
     (pin "1")
+  )
+  (symbol (lib_id "Connector:Screw_Terminal_01x04") (at 113.03 38.1 0) (mirror x) (unit 1)
+    (in_bom yes) (on_board yes) (fields_autoplaced)
+    (property "Reference" "J5" (id 0) (at 113.03 26.67 0))
+    (property "Value" "Screw_Terminal_01x04" (id 1) (at 113.03 29.21 0))
+    (property "Footprint" "TerminalBlock_Phoenix:TerminalBlock_Phoenix_MPT-0,5-4-2.54_1x04_P2.54mm_Horizontal" (id 2) (at 113.03 38.1 0)
+      (effects (font (size 1.27 1.27)) hide)
+    )
+    (property "Datasheet" "~" (id 3) (at 113.03 38.1 0)
+      (effects (font (size 1.27 1.27)) hide)
+    )
+    (pin "1")
+    (pin "2")
+    (pin "3")
+    (pin "4")
   )
   (symbol (lib_id "Device:R") (at 64.77 60.96 0) (unit 1)
@@
     (pin "2")
   )
-  (symbol (lib_id "Connector_Generic:Conn_01x02") (at 80.01 22.86 0) (unit 1)
-    (in_bom yes) (on_board yes) (fields_autoplaced)
-    (property "Reference" "J11" (id 0) (at 82.55 22.8599 0)
-      (effects (font (size 1.27 1.27)) (justify left))
-    )
-    (property "Value" "Conn_01x02" (id 1) (at 82.55 25.3999 0)
-      (effects (font (size 1.27 1.27)) (justify left))
-    )
-    (property "Footprint" "TerminalBlock_Phoenix:TerminalBlock_Phoenix_PT-1,5-2-5.0-H_1x02_P5.00mm_Horizontal" (id 2) (at 80.01 22.86 0)
-      (effects (font (size 1.27 1.27)) hide)
-    )
-    (property "Datasheet" "~" (id 3) (at 80.01 22.86 0)
-      (effects (font (size 1.27 1.27)) hide)
-    )
-    (pin "1")
-    (pin "2")
-  )
   (symbol (lib_id "Device:R") (at 64.77 105.41 0) (unit 1)
     (in_bom yes) (on_board yes) (fields_autoplaced)
@@
       (effects (font (size 1.27 1.27)) hide)
     )
-    (pin "1")
-    (pin "2")
-  )
-  (symbol (lib_id "Connector_Generic:Conn_01x02") (at 80.01 80.01 0) (unit 1)
-    (in_bom yes) (on_board yes) (fields_autoplaced)
-    (property "Reference" "J12" (id 0) (at 82.55 80.0099 0)
-      (effects (font (size 1.27 1.27)) (justify left))
-    )
-    (property "Value" "Conn_01x02" (id 1) (at 82.55 82.5499 0)
-      (effects (font (size 1.27 1.27)) (justify left))
-    )
-    (property "Footprint" "TerminalBlock_Phoenix:TerminalBlock_Phoenix_PT-1,5-2-5.0-H_1x02_P5.00mm_Horizontal" (id 2) (at 80.01 80.01 0)
-      (effects (font (size 1.27 1.27)) hide)
-    )
-    (property "Datasheet" "~" (id 3) (at 80.01 80.01 0)
-      (effects (font (size 1.27 1.27)) hide)
-    )

Commit message: Lots of adjustments, 3 way I2C bus selection, SMD diodes
Parts:
- D1, D2: footprint Diode_THT:D_DO-41_SOD81_P2.54mm_Vertical_AnodeUp -> Diode_SMD:D_SOD-323_HandSoldering
Changed lines of the file:
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@@
       (effects (font (size 1.27 1.27)) (justify left))
     )
-    (property "Footprint" "Diode_THT:D_DO-41_SOD81_P2.54mm_Vertical_AnodeUp" (id 2) (at 54.61 118.11 0)
+    (property "Footprint" "Diode_SMD:D_SOD-323_HandSoldering" (id 2) (at 54.61 118.11 0)
       (effects (font (size 1.27 1.27)) hide)
     )
@@
       (effects (font (size 1.27 1.27)) (justify left))
     )
-    (property "Footprint" "Diode_THT:D_DO-41_SOD81_P2.54mm_Vertical_AnodeUp" (id 2) (at 54.61 60.96 0)
+    (property "Footprint" "Diode_SMD:D_SOD-323_HandSoldering" (id 2) (at 54.61 60.96 0)
       (effects (font (size 1.27 1.27)) hide)
     )

Commit message: Change diode footprint
Parts:
- D1, D2: value 3v3 -> BZX384-C3V3,115; footprint Diode_SMD:D_SOD-323_HandSoldering -> Diode_SMD:D_SOD-323
Other:
- moved on the sheet: R10, R11, R12, R9
