File: Motherboard/motherboard_2022_2023/hdmi 2.kicad_sch (KiCad schematic)
At the start: 2 parts, among them J13 Conn_01x22_Shielded, J14 HDMI_C_1.4

Commit message: Add mousebite
Parts:
- removed J13: Conn_01x22_Shielded, custom-footprints:MOLEX 22 Pin FPC 54548-2271, symbol Connector_Generic_Shielded:Conn_01x22_Shielded
- removed J14: HDMI_C_1.4, custom-footprints:WURTH_685119136923, symbol Connector:HDMI_C_1.4
- added H7: MountingHole, custom-footprints:mousebite, symbol Mechanical:MountingHole
- added J15: (no value), symbol Connector_Generic_Shielded:Conn_01x22_Shielded
- added J16: (no value), symbol Connector:HDMI_C_1.4
Connections:
- net CAM_3V3: now also J15.1 (Pin_1), J16.18 (+5V)
- net CAM_GND: now also J15.10 (Pin_10), J15.13 (Pin_13), J15.16 (Pin_16), J15.19 (Pin_19), J15.22 (Pin_22), J15.4 (Pin_4), J15.7 (Pin_7), J15.SH (Shield), J16.1 (D2S), J16.10 (CKS), J16.13 (GND), J16.4 (D1S), J16.7 (D0S), J16.SH
- net CAM_SCL: now also J15.3 (Pin_3), J16.15 (SCL)
- net CAM_SDA: now also J15.2 (Pin_2), J16.16 (SDA)
- net D0+: now also J15.21 (Pin_21), J16.2 (D2+)
- net D0-: now also J15.20 (Pin_20), J16.3 (D2-)
- net D1+: now also J15.18 (Pin_18), J16.5 (D1+)
- net D1-: now also J15.17 (Pin_17), J16.6 (D1-)
- net DC+: now also J15.15 (Pin_15), J16.8 (D0+)
- net DC-: now also J15.14 (Pin_14), J16.9 (D0-)
- net GPIO0: now also J15.6 (Pin_6), J16.11 (CK+)
- net GPIO1: now also J15.5 (Pin_5), J16.12 (CK-)
Changed lines of the file:
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@@
   (junction (at 81.28 67.31) (diameter 0) (color 0 0 0 0)
-  )
-  (junction (at 81.28 111.76) (diameter 0) (color 0 0 0 0)
   )
   (junction (at 137.16 109.22) (diameter 0) (color 0 0 0 0)
@@
     (stroke (width 0) (type default) (color 0 0 0 0))
   )
-  (wire (pts (xy 71.12 110.49) (xy 71.12 111.76))
-    (stroke (width 0) (type default) (color 0 0 0 0))
-  )
   (wire (pts (xy 121.92 86.36) (xy 111.76 86.36))
     (stroke (width 0) (type default) (color 0 0 0 0))
@@
     (stroke (width 0) (type default) (color 0 0 0 0))
   )
-  (wire (pts (xy 71.12 111.76) (xy 81.28 111.76))
-    (stroke (width 0) (type default) (color 0 0 0 0))
-  )
   (wire (pts (xy 76.2 64.77) (xy 95.25 64.77))
     (stroke (width 0) (type default) (color 0 0 0 0))
@@
     (stroke (width 0) (type default) (color 0 0 0 0))
   )
+  (wire (pts (xy 71.12 46.99) (xy 71.12 34.29))
+    (stroke (width 0) (type default) (color 0 0 0 0))
+  )
   (wire (pts (xy 121.92 71.12) (xy 111.76 71.12))
     (stroke (width 0) (type default) (color 0 0 0 0))
@@
   (label "D1-" (at 111.76 66.04 0)
     (effects (font (size 1.27 1.27)) (justify left bottom))
+  )
+  (label "CAM_GND" (at 71.12 34.29 270)
+    (effects (font (size 1.27 1.27)) (justify right bottom))
   )
   (label "D1-" (at 95.25 64.77 180)
@@
   (symbol (lib_id "Connector:HDMI_C_1.4") (at 132.08 78.74 0) (unit 1)
     (in_bom yes) (on_board yes) (fields_autoplaced)
-    (property "Reference" "J14" (id 0) (at 143.51 77.4699 0)
+    (property "Reference" "J16" (id 0) (at 143.51 77.4699 0)
       (effects (font (size 1.27 1.27)) (justify left))
     )
-    (property "Value" "HDMI_C_1.4" (id 1) (at 143.51 80.0099 0)
+    (property "Value" "" (id 1) (at 143.51 80.0099 0)
       (effects (font (size 1.27 1.27)) (justify left))
     )
-    (property "Footprint" "custom-footprints:WURTH_685119136923" (id 2) (at 132.715 78.74 0)
+    (property "Footprint" "" (id 2) (at 132.715 78.74 0)
       (effects (font (size 1.27 1.27)) hide)
     )
@@
     (pin "SH")
   )
-  (symbol (lib_id "Connector_Generic_Shielded:Conn_01x22_Shielded") (at 71.12 77.47 0) (mirror y) (unit 1)
+  (symbol (lib_id "Mechanical:MountingHole") (at 97.79 35.56 0) (unit 1)
     (in_bom yes) (on_board yes) (fields_autoplaced)
-    (property "Reference" "J13" (id 0) (at 71.12 45.72 0))
-    (property "Value" "Conn_01x22_Shielded" (id 1) (at 71.12 48.26 0))
-    (property "Footprint" "custom-footprints:MOLEX 22 Pin FPC 54548-2271" (id 2) (at 71.12 77.47 0)
-      (effects (font (size 1.27 1.27)) hide)
-    )
-    (property "Datasheet" "~" (id 3) (at 71.12 77.47 0)
-      (effects (font (size 1.27 1.27)) hide)
-    )
+    (property "Reference" "H7" (id 0) (at 95.25 34.2899 0)
+      (effects (font (size 1.27 1.27)) (justify right))
+    )
+    (property "Value" "MountingHole" (id 1) (at 95.25 36.8299 0)
+      (effects (font (size 1.27 1.27)) (justify right))
+    )
+    (property "Footprint" "custom-footprints:mousebite" (id 2) (at 97.79 35.56 0)
+      (effects (font (size 1.27 1.27)) hide)
+    )
+    (property "Datasheet" "~" (id 3) (at 97.79 35.56 0)
+      (effects (font (size 1.27 1.27)) hide)
+    )
+  )
+  (symbol (lib_id "Connector_Generic_Shielded:Conn_01x22_Shielded") (at 71.12 80.01 180) (unit 1)
+    (in_bom yes) (on_board yes) (fields_autoplaced)
+    (property "Reference" "J15" (id 0) (at 68.58 77.4699 0)
+      (effects (font (size 1.27 1.27)) (justify left))
+    )
+    (property "Value" "" (id 1) (at 68.58 80.0099 0)
+      (effects (font (size 1.27 1.27)) (justify left))
+    )
+    (property "Footprint" "" (id 2) (at 71.12 80.01 0)
+      (effects (font (size 1.27 1.27)) hide)
+    )
+    (property "Datasheet" "~" (id 3) (at 71.12 80.01 0)
+      (effects (font (size 1.27 1.27)) hide)
+    )
