File: Motherboard/motherboard_2022_2023/hdmi_to_csi.kicad_pcb (KiCad board)
At the start: 2 copper layers, 29.2 x 17.1 mm, 4 parts, among them J15 Conn_01x22_Shielded, J16 HDMI_C_1.4

Commit message: Fixed Daughterboard
Parts:
- J1: renamed from J15; value Conn_01x22_Shielded -> ~
- J2: renamed from J16; value HDMI_C_1.4 -> ~
- renumbered H6 to H1, H5 to H2
Connections:
- J1 pad 1: (no net) -> /CAM_3V3
- J1 pad 10: (no net) -> /CAM_GND
- J1 pad 11: (no net) -> unconnected-(J1-Pad11)
- J1 pad 12: (no net) -> unconnected-(J1-Pad12)
- J1 pad 13: (no net) -> /CAM_GND
- J1 pad 14: (no net) -> /DC-
- J1 pad 15: (no net) -> /DC+
- J1 pad 16: (no net) -> /CAM_GND
- J1 pad 17: (no net) -> /D1-
- J1 pad 18: (no net) -> /D1+
- J1 pad 19: (no net) -> /CAM_GND
- J1 pad 2: (no net) -> /CAM_SDA
- J1 pad 20: (no net) -> /D0-
- J1 pad 21: (no net) -> /D0+
- J1 pad 22: (no net) -> /CAM_GND
- J1 pad 3: (no net) -> /CAM_SCL
- J1 pad 4: (no net) -> /CAM_GND
- J1 pad 5: (no net) -> /GPIO1
- J1 pad 6: (no net) -> /GPIO0
- J1 pad 7: (no net) -> /CAM_GND
- J1 pad 8: (no net) -> unconnected-(J1-Pad8)
- J1 pad 9: (no net) -> unconnected-(J1-Pad9)
- J1 pad SH: (no net) -> /CAM_GND
- J2 pad 1: (no net) -> /CAM_GND
- J2 pad 10: (no net) -> /CAM_GND
- J2 pad 11: (no net) -> /GPIO0
- J2 pad 12: (no net) -> /GPIO1
- J2 pad 13: (no net) -> /CAM_GND
- J2 pad 14: (no net) -> unconnected-(J2-Pad14)
- J2 pad 15: (no net) -> /CAM_SCL
- J2 pad 16: (no net) -> /CAM_SDA
- J2 pad 17: (no net) -> unconnected-(J2-Pad17)
- J2 pad 18: (no net) -> /CAM_3V3
- J2 pad 19: (no net) -> unconnected-(J2-Pad19)
- J2 pad 2: (no net) -> /D0+
- J2 pad 3: (no net) -> /D0-
- J2 pad 4: (no net) -> /CAM_GND
- J2 pad 5: (no net) -> /D1+
- J2 pad 6: (no net) -> /D1-
- J2 pad 7: (no net) -> /CAM_GND
- J2 pad 8: (no net) -> /DC+
- J2 pad 9: (no net) -> /DC-
- J2 pad SH: (no net) -> /CAM_GND
Routing:
- net (no net): track 61.8 -> 0.00 mm, vias 11 -> 0
- net /CAM_SDA: track 0.00 -> 6.18 mm, vias 0 -> 1
- net /CAM_3V3: track 0.00 -> 6.15 mm, vias 0 -> 1
- net /GPIO1: track 0.00 -> 6.02 mm, vias 0 -> 1
- net /GPIO0: track 0.00 -> 5.98 mm, vias 0 -> 1
- net /CAM_SCL: track 0.00 -> 5.94 mm, vias 0 -> 1
- net /D1-: track 0.00 -> 5.46 mm, vias 0 -> 1
- net /D1+: track 0.00 -> 5.46 mm, vias 0 -> 1
- net /DC-: track 0.00 -> 5.34 mm, vias 0 -> 1
- net /D0+: track 0.00 -> 5.20 mm, vias 0 -> 1
- net /DC+: track 0.00 -> 5.09 mm, vias 0 -> 1
- net /D0-: track 0.00 -> 4.96 mm, vias 0 -> 1
- added copper zone on B.Cu, net /CAM_GND
- added copper zone on F.Cu, net /CAM_GND
- removed copper zone on B.Cu, net (none)
- removed copper zone on F.Cu, net (none)
