File: Motherboard/motherboard_2022_2023/hdmi_to_csi.kicad_sch (KiCad schematic)
At the start: 3 parts

Commit message: Moved CSI to HDMI to own PCB
Parts:
- added H1: MountingHole, MountingHole:MountingHole_2.5mm, symbol Mechanical:MountingHole
- J15, J16: value (none) -> ~
- renumbered H7 to H2
Other:
- title: (none) -> HDMI to CSI Conversion (Reversed)
- moved on the sheet: H2
Changed lines of the file:
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@@
 (kicad_sch (version 20211123) (generator eeschema)
   (paper "A4")
+  (title_block
+    (title "HDMI to CSI Conversion (Reversed)")
+    (date "2022-11-28")
+    (rev "1.0")
+  )
   (junction (at 81.28 97.79) (diameter 0) (color 0 0 0 0)
   )
@@
       (effects (font (size 1.27 1.27)) (justify left))
     )
-    (property "Value" "" (id 1) (at 143.51 80.0099 0)
+    (property "Value" "~" (id 1) (at 143.51 80.0099 0)
       (effects (font (size 1.27 1.27)) (justify left))
     )
@@
     (pin "SH")
   )
-  (symbol (lib_id "Mechanical:MountingHole") (at 97.79 35.56 0) (unit 1)
+  (symbol (lib_id "Mechanical:MountingHole") (at 107.95 38.1 0) (unit 1)
     (in_bom yes) (on_board yes) (fields_autoplaced)
-    (property "Reference" "H7" (id 0) (at 95.25 34.2899 0)
+    (property "Reference" "H1" (id 0) (at 105.41 36.8299 0)
       (effects (font (size 1.27 1.27)) (justify right))
     )
-    (property "Value" "MountingHole" (id 1) (at 95.25 36.8299 0)
+    (property "Value" "MountingHole" (id 1) (at 105.41 39.3699 0)
       (effects (font (size 1.27 1.27)) (justify right))
     )
-    (property "Footprint" "custom-footprints:mousebite" (id 2) (at 97.79 35.56 0)
-      (effects (font (size 1.27 1.27)) hide)
-    )
-    (property "Datasheet" "~" (id 3) (at 97.79 35.56 0)
+    (property "Footprint" "MountingHole:MountingHole_2.5mm" (id 2) (at 107.95 38.1 0)
+      (effects (font (size 1.27 1.27)) hide)
+    )
+    (property "Datasheet" "~" (id 3) (at 107.95 38.1 0)
+      (effects (font (size 1.27 1.27)) hide)
+    )
+  )
+  (symbol (lib_id "Mechanical:MountingHole") (at 110.49 127 0) (unit 1)
+    (in_bom yes) (on_board yes) (fields_autoplaced)
+    (property "Reference" "H2" (id 0) (at 113.03 125.7299 0)
+      (effects (font (size 1.27 1.27)) (justify left))
+    )
+    (property "Value" "MountingHole" (id 1) (at 113.03 128.2699 0)
+      (effects (font (size 1.27 1.27)) (justify left))
+    )
+    (property "Footprint" "custom-footprints:mousebite" (id 2) (at 110.49 127 0)
+      (effects (font (size 1.27 1.27)) hide)
+    )
+    (property "Datasheet" "~" (id 3) (at 110.49 127 0)
       (effects (font (size 1.27 1.27)) hide)
     )
@@
       (effects (font (size 1.27 1.27)) (justify left))
     )
-    (property "Value" "" (id 1) (at 68.58 80.0099 0)
+    (property "Value" "~" (id 1) (at 68.58 80.0099 0)
       (effects (font (size 1.27 1.27)) (justify left))
     )
@@
     (pin "SH")
   )
+  (sheet_instances
+    (path "/" (page "1"))
+  )
+  (symbol_instances
+    (path "/6f88ccac-dcd9-4e98-b2bc-4b7858a309c8"
+      (reference "H1") (unit 1) (value "MountingHole") (footprint "MountingHole:MountingHole_2.5mm")
+    )
+    (path "/bc950924-1296-4adb-a209-9b9be0edae2e"
+      (reference "H2") (unit 1) (value "MountingHole") (footprint "custom-footprints:mousebite")
+    )
+    (path "/e046bb90-a8e9-4e7f-8aa0-c8908f4f92d0"
+      (reference "J15") (unit 1) (value "~") (footprint "")
+    )
+    (path "/1cd00081-e313-451c-acb4-77e1c887fa82"
+      (reference "J16") (unit 1) (value "~") (footprint "")
+    )
+  )
 )

Commit message: Fixed Daughterboard
Parts:
- H1: renamed from H2; footprint custom-footprints:mousebite -> MountingHole:MountingHole_3.2mm_M3
- H2: renamed from H1; footprint MountingHole:MountingHole_2.5mm -> MountingHole:MountingHole_3.2mm_M3
- J1: renamed from J15; footprint (none) -> custom-footprints:MOLEX 22 Pin FPC 54548-2271
- J2: renamed from J16; footprint (none) -> custom-footprints:WURTH_685119136923
Other:
- moved on the sheet: H1
Changed lines of the file:
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@@
   (symbol (lib_id "Connector:HDMI_C_1.4") (at 132.08 78.74 0) (unit 1)
     (in_bom yes) (on_board yes) (fields_autoplaced)
-    (property "Reference" "J16" (id 0) (at 143.51 77.4699 0)
+    (property "Reference" "J2" (id 0) (at 143.51 77.4699 0)
       (effects (font (size 1.27 1.27)) (justify left))
     )
@@
       (effects (font (size 1.27 1.27)) (justify left))
     )
-    (property "Footprint" "" (id 2) (at 132.715 78.74 0)
+    (property "Footprint" "custom-footprints:WURTH_685119136923" (id 2) (at 132.715 78.74 0)
       (effects (font (size 1.27 1.27)) hide)
     )
@@
   (symbol (lib_id "Mechanical:MountingHole") (at 107.95 38.1 0) (unit 1)
     (in_bom yes) (on_board yes) (fields_autoplaced)
-    (property "Reference" "H1" (id 0) (at 105.41 36.8299 0)
+    (property "Reference" "H2" (id 0) (at 105.41 36.8299 0)
       (effects (font (size 1.27 1.27)) (justify right))
     )
@@
       (effects (font (size 1.27 1.27)) (justify right))
     )
-    (property "Footprint" "MountingHole:MountingHole_2.5mm" (id 2) (at 107.95 38.1 0)
+    (property "Footprint" "MountingHole:MountingHole_3.2mm_M3" (id 2) (at 107.95 38.1 0)
       (effects (font (size 1.27 1.27)) hide)
     )
@@
     )
   )
-  (symbol (lib_id "Mechanical:MountingHole") (at 110.49 127 0) (unit 1)
+  (symbol (lib_id "Mechanical:MountingHole") (at 105.41 120.65 0) (unit 1)
     (in_bom yes) (on_board yes) (fields_autoplaced)
-    (property "Reference" "H2" (id 0) (at 113.03 125.7299 0)
+    (property "Reference" "H1" (id 0) (at 107.95 119.3799 0)
       (effects (font (size 1.27 1.27)) (justify left))
     )
-    (property "Value" "MountingHole" (id 1) (at 113.03 128.2699 0)
+    (property "Value" "MountingHole" (id 1) (at 107.95 121.9199 0)
       (effects (font (size 1.27 1.27)) (justify left))
     )
-    (property "Footprint" "custom-footprints:mousebite" (id 2) (at 110.49 127 0)
+    (property "Footprint" "MountingHole:MountingHole_3.2mm_M3" (id 2) (at 105.41 120.65 0)
       (effects (font (size 1.27 1.27)) hide)
     )
-    (property "Datasheet" "~" (id 3) (at 110.49 127 0)
+    (property "Datasheet" "~" (id 3) (at 105.41 120.65 0)
       (effects (font (size 1.27 1.27)) hide)
     )
@@
   (symbol (lib_id "Connector_Generic_Shielded:Conn_01x22_Shielded") (at 71.12 80.01 180) (unit 1)
     (in_bom yes) (on_board yes) (fields_autoplaced)
-    (property "Reference" "J15" (id 0) (at 68.58 77.4699 0)
+    (property "Reference" "J1" (id 0) (at 68.58 77.4699 0)
       (effects (font (size 1.27 1.27)) (justify left))
     )
@@
       (effects (font (size 1.27 1.27)) (justify left))
     )
-    (property "Footprint" "" (id 2) (at 71.12 80.01 0)
+    (property "Footprint" "custom-footprints:MOLEX 22 Pin FPC 54548-2271" (id 2) (at 71.12 80.01 0)
       (effects (font (size 1.27 1.27)) hide)
     )
@@
   )
   (symbol_instances
+    (path "/bc950924-1296-4adb-a209-9b9be0edae2e"
+      (reference "H1") (unit 1) (value "MountingHole") (footprint "MountingHole:MountingHole_3.2mm_M3")
+    )
     (path "/6f88ccac-dcd9-4e98-b2bc-4b7858a309c8"
-      (reference "H1") (unit 1) (value "MountingHole") (footprint "MountingHole:MountingHole_2.5mm")
-    )
-    (path "/bc950924-1296-4adb-a209-9b9be0edae2e"
-      (reference "H2") (unit 1) (value "MountingHole") (footprint "custom-footprints:mousebite")
+      (reference "H2") (unit 1) (value "MountingHole") (footprint "MountingHole:MountingHole_3.2mm_M3")
     )
     (path "/e046bb90-a8e9-4e7f-8aa0-c8908f4f92d0"
-      (reference "J15") (unit 1) (value "~") (footprint "")
+      (reference "J1") (unit 1) (value "~") (footprint "custom-footprints:MOLEX 22 Pin FPC 54548-2271")
     )
     (path "/1cd00081-e313-451c-acb4-77e1c887fa82"
-      (reference "J16") (unit 1) (value "~") (footprint "")
+      (reference "J2") (unit 1) (value "~") (footprint "custom-footprints:WURTH_685119136923")
     )
   )
