File: Motherboard/motherboard_2022_2023/hdmi.kicad_sch (KiCad schematic)
At the start: 2 parts, among them J13 Conn_01x22_Shielded, J14 HDMI_C_1.4

Commit message: Added Title
Other:
- company: (none) -> Rose Rocketry
- title: (none) -> CSI-to-HDMI Motherboard
Changed lines of the file:
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@@
 (kicad_sch (version 20211123) (generator eeschema)
   (paper "A4")
+  (title_block
+    (title "CSI-to-HDMI Motherboard")
+    (date "2022-11-30")
+    (company "Rose Rocketry")
+    (comment 1 "Author: Evelyn Gordon")
+  )
   (junction (at 81.28 97.79) (diameter 0) (color 0 0 0 0)
   )

Commit message: Added Images to Title Blocks
Other:
- company: Rose Rocketry -> Rose-Hulman Institute of Technology

Commit message: Fix flipped FFC connector
Connections:
- net CAM_3V3: now also J13.1 (Pin_1); no longer J13.22 (Pin_22)
- net CAM_GND: now also J13.22 (Pin_22); no longer J13.1 (Pin_1)
- net CAM_SCL: now also J13.3 (Pin_3); no longer J13.20 (Pin_20)
- net CAM_SDA: now also J13.2 (Pin_2); no longer J13.21 (Pin_21)
- net D0+: now also J13.21 (Pin_21); no longer J13.2 (Pin_2)
- net D0-: now also J13.20 (Pin_20); no longer J13.3 (Pin_3)
- net D1+: now also J13.18 (Pin_18); no longer J13.5 (Pin_5)
- net D1-: now also J13.17 (Pin_17); no longer J13.6 (Pin_6)
- net DC+: now also J13.15 (Pin_15); no longer J13.8 (Pin_8)
- net DC-: now also J13.14 (Pin_14); no longer J13.9 (Pin_9)
- net GPIO0: now also J13.6 (Pin_6); no longer J13.17 (Pin_17)
- net GPIO1: now also J13.5 (Pin_5); no longer J13.18 (Pin_18)
Other:
- moved on the sheet: J13
Changed lines of the file:
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@@
     (comment 2 "For Rose Rocketry")
   )
+  (junction (at 81.28 52.07) (diameter 0) (color 0 0 0 0)
+  )
   (junction (at 81.28 97.79) (diameter 0) (color 0 0 0 0)
   )
@@
   )
   (junction (at 81.28 67.31) (diameter 0) (color 0 0 0 0)
-  )
-  (junction (at 81.28 111.76) (diameter 0) (color 0 0 0 0)
   )
   (junction (at 137.16 109.22) (diameter 0) (color 0 0 0 0)
@@
   (no_connect (at 121.92 93.98))
   (no_connect (at 76.2 85.09))
+  (wire (pts (xy 81.28 46.99) (xy 81.28 52.07))
+    (stroke (width 0) (type default) (color 0 0 0 0))
+  )
   (wire (pts (xy 139.7 109.22) (xy 137.16 109.22))
     (stroke (width 0) (type default) (color 0 0 0 0))
@@
     (stroke (width 0) (type default) (color 0 0 0 0))
   )
-  (wire (pts (xy 71.12 110.49) (xy 71.12 111.76))
-    (stroke (width 0) (type default) (color 0 0 0 0))
-  )
   (wire (pts (xy 121.92 86.36) (xy 111.76 86.36))
     (stroke (width 0) (type default) (color 0 0 0 0))
@@
     (stroke (width 0) (type default) (color 0 0 0 0))
   )
-  (wire (pts (xy 71.12 111.76) (xy 81.28 111.76))
-    (stroke (width 0) (type default) (color 0 0 0 0))
-  )
   (wire (pts (xy 76.2 64.77) (xy 95.25 64.77))
     (stroke (width 0) (type default) (color 0 0 0 0))
@@
   )
   (wire (pts (xy 81.28 97.79) (xy 81.28 111.76))
+    (stroke (width 0) (type default) (color 0 0 0 0))
+  )
+  (wire (pts (xy 71.12 46.99) (xy 81.28 46.99))
     (stroke (width 0) (type default) (color 0 0 0 0))
   )
@@
     (pin "SH")
   )
-  (symbol (lib_id "Connector_Generic_Shielded:Conn_01x22_Shielded") (at 71.12 77.47 0) (mirror y) (unit 1)
+  (symbol (lib_id "Connector_Generic_Shielded:Conn_01x22_Shielded") (at 71.12 80.01 180) (unit 1)
     (in_bom yes) (on_board yes) (fields_autoplaced)
-    (property "Reference" "J13" (id 0) (at 71.12 45.72 0))
-    (property "Value" "Conn_01x22_Shielded" (id 1) (at 71.12 48.26 0))
-    (property "Footprint" "custom-footprints:MOLEX 22 Pin FPC 54548-2271" (id 2) (at 71.12 77.47 0)
+    (property "Reference" "J13" (id 0) (at 68.58 77.4699 0)
+      (effects (font (size 1.27 1.27)) (justify left))
+    )
+    (property "Value" "Conn_01x22_Shielded" (id 1) (at 68.58 80.0099 0)
+      (effects (font (size 1.27 1.27)) (justify left))
+    )
+    (property "Footprint" "custom-footprints:MOLEX 22 Pin FPC 54548-2271" (id 2) (at 71.12 80.01 0)
       (effects (font (size 1.27 1.27)) hide)
     )
-    (property "Datasheet" "~" (id 3) (at 71.12 77.47 0)
+    (property "Datasheet" "~" (id 3) (at 71.12 80.01 0)
       (effects (font (size 1.27 1.27)) hide)
     )
