File: Motherboard/motherboard_2022_2023/motherboard_2022_2023.kicad_pcb (KiCad board)
At the start: 2 copper layers, 139.7 x 50.8 mm, 69 parts, among them J1 Conn_01x02_Female, J11 Conn_01x02, J12 Conn_01x02, J13 Conn_01x22_Shielded, J14 HDMI_C_1.4, J2 Raspberry_Pi_2_3, J3 Conn_02x04_Counter_Clockwise, J4 STEMMA QT, Q1 AO4838, SW1 SHUTDOWN, U1 XBee_THT, U3 PCA9685PW, U4 MPL3115A2, U5 TPS56424x, U6 SAM-M8Q, U7 MPU-6050, U8 MCP3004

Commit message: Fix SDA/SCL swapped on MPU6050 and MPL3115
Connections:
- U4 pad 7: /SCL -> /SDA
- U4 pad 8: /SDA -> /SCL
- U7 pad 23: /SDA -> /SCL
- U7 pad 24: /SCL -> /SDA
Routing:
- net /SCL: track 140.9 -> 133.0 mm, vias 3 -> 5
- net /SDA: track 141.5 -> 137.3 mm, vias 3 -> 5
- net +3V3: track 264.5 -> 261.6 mm
- net GND: vias 38 -> 37

Commit message: Fix flipped FFC connector
Parts:
- moved J13 12.5 mm to (155.3, 110.8)
- moved J14 5.52 mm to (166.5, 119.8)
Connections:
- J13 pad 1: /HDMI CSI Conversion/CAM_GND -> /HDMI CSI Conversion/CAM_3V3
- J13 pad 14: unconnected-(J13-Pad14) -> /HDMI CSI Conversion/DC-
- J13 pad 15: unconnected-(J13-Pad15) -> /HDMI CSI Conversion/DC+
- J13 pad 17: /HDMI CSI Conversion/GPIO0 -> /HDMI CSI Conversion/D1-
- J13 pad 18: /HDMI CSI Conversion/GPIO1 -> /HDMI CSI Conversion/D1+
- J13 pad 2: /HDMI CSI Conversion/D0+ -> /HDMI CSI Conversion/CAM_SDA
- J13 pad 20: /HDMI CSI Conversion/CAM_SCL -> /HDMI CSI Conversion/D0-
- J13 pad 21: /HDMI CSI Conversion/CAM_SDA -> /HDMI CSI Conversion/D0+
- J13 pad 22: /HDMI CSI Conversion/CAM_3V3 -> /HDMI CSI Conversion/CAM_GND
- J13 pad 3: /HDMI CSI Conversion/D0- -> /HDMI CSI Conversion/CAM_SCL
- J13 pad 5: /HDMI CSI Conversion/D1+ -> /HDMI CSI Conversion/GPIO1
- J13 pad 6: /HDMI CSI Conversion/D1- -> /HDMI CSI Conversion/GPIO0
- J13 pad 8: /HDMI CSI Conversion/DC+ -> unconnected-(J13-Pad8)
- J13 pad 9: /HDMI CSI Conversion/DC- -> unconnected-(J13-Pad9)
Routing:
- net /HDMI CSI Conversion/CAM_GND: track 141.0 -> 191.0 mm
- net /HDMI CSI Conversion/D0+: track 7.24 -> 22.5 mm
- net /HDMI CSI Conversion/D0-: track 7.82 -> 21.9 mm
- net /HDMI CSI Conversion/D1+: track 9.23 -> 20.5 mm
- net /HDMI CSI Conversion/D1-: track 9.81 -> 19.9 mm
- net /HDMI CSI Conversion/CAM_3V3: track 18.8 -> 10.7 mm
- net /HDMI CSI Conversion/DC+: track 11.2 -> 18.5 mm
- net /HDMI CSI Conversion/CAM_SDA: track 18.0 -> 11.6 mm
- net /HDMI CSI Conversion/DC-: track 11.8 -> 17.9 mm
- net /HDMI CSI Conversion/CAM_SCL: track 17.3 -> 12.2 mm
- net /HDMI CSI Conversion/GPIO1: track 15.8 -> 13.7 mm
- net /HDMI CSI Conversion/GPIO0: track 15.2 -> 14.4 mm

Commit message: Remove unused pullup
Parts:
- removed R1: 10k, Resistor_SMD:R_0603_1608Metric
Routing:
- net +3V3: track 261.6 -> 256.2 mm
- net /SHUTDOWN: track 17.8 -> 16.5 mm
Changed lines of the file:
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@@
-    )
-  )
-  (footprint "Resistor_SMD:R_0603_1608Metric" (layer "F.Cu")
-    (at 148.995562 103.009695 180)
-    (descr "Resistor SMD 0603 (1608 Metric), square (rectangular) end terminal, IPC_7351 nominal, (Body size source: IPC-SM-782 page 72, https://www.pcb-3d.com/wordpress/wp-content/uploads/ipc-sm-782a_amendment_1_and_2.pdf), generated with kicad-footprint-generator")
-    (tags "resistor")
-    (property "Sheetfile" "motherboard_2022_2023.kicad_sch")
-    (property "Sheetname" "")
-    (attr smd)
-    (fp_text reference "R1" (at 0 -1.43) (layer "F.SilkS")
-      (effects (font (size 1 1) (thickness 0.15)))
-    )
-    (fp_text value "10k" (at 0 1.43) (layer "F.Fab")
-      (effects (font (size 1 1) (thickness 0.15)))
-    )
-    (fp_text user "${REFERENCE}" (at 0 0) (layer "F.Fab")
-      (effects (font (size 0.4 0.4) (thickness 0.06)))
-    )
-    (fp_line (start -0.237258 -0.5225) (end 0.237258 -0.5225) (layer "F.SilkS") (width 0.12))
-    (fp_line (start -0.237258 0.5225) (end 0.237258 0.5225) (layer "F.SilkS") (width 0.12))
-    (fp_line (start -1.48 -0.73) (end 1.48 -0.73) (layer "F.CrtYd") (width 0.05))
-    (fp_line (start 1.48 0.73) (end -1.48 0.73) (layer "F.CrtYd") (width 0.05))
-    (fp_line (start 1.48 -0.73) (end 1.48 0.73) (layer "F.CrtYd") (width 0.05))
-    (fp_line (start -1.48 0.73) (end -1.48 -0.73) (layer "F.CrtYd") (width 0.05))
-    (fp_line (start 0.8 -0.4125) (end 0.8 0.4125) (layer "F.Fab") (width 0.1))
-    (fp_line (start -0.8 0.4125) (end -0.8 -0.4125) (layer "F.Fab") (width 0.1))
-    (fp_line (start 0.8 0.4125) (end -0.8 0.4125) (layer "F.Fab") (width 0.1))
-    (fp_line (start -0.8 -0.4125) (end 0.8 -0.4125) (layer "F.Fab") (width 0.1))
-    (pad "1" smd roundrect (at -0.825 0 180) (size 0.8 0.95) (layers "F.Cu" "F.Paste" "F.Mask") (roundrect_rratio 0.25)
-      (net 8 "/SHUTDOWN") (pintype "passive"))
-    (pad "2" smd roundrect (at 0.825 0 180) (size 0.8 0.95) (layers "F.Cu" "F.Paste" "F.Mask") (roundrect_rratio 0.25)
-      (net 5 "+3V3") (pintype "passive"))
-    (model "${KICAD6_3DMODEL_DIR}/Resistor_SMD.3dshapes/R_0603_1608Metric.wrl"
-      (offset (xyz 0 0 0))
-      (scale (xyz 1 1 1))
-      (rotate (xyz 0 0 0))
     )
   )
@@
   (segment (start 144.677562 100.145695) (end 144.677562 113.169695) (width 1) (layer "F.Cu") (net 5))
   (segment (start 180.874562 101.741695) (end 180.874562 112.876438) (width 0.2) (layer "F.Cu") (net 5))
-  (segment (start 144.677562 101.358695) (end 144.677562 100.145695) (width 0.25) (layer "F.Cu") (net 5))
-  (segment (start 148.170562 103.009695) (end 146.328562 103.009695) (width 0.25) (layer "F.Cu") (net 5))
   (segment (start 133.856562 84.272195) (end 133.856562 84.960736) (width 0.25) (layer "F.Cu") (net 5))
   (segment (start 137 88) (end 136.967562 87.967562) (width 0.25) (layer "F.Cu") (net 5))
@@
   (segment (start 97.306562 120.658695) (end 97.306562 124.345695) (width 1) (layer "F.Cu") (net 5))
   (segment (start 80.01 113.538) (end 81.038695 114.566695) (width 0.25) (layer "F.Cu") (net 5))
-  (segment (start 146.328562 103.009695) (end 144.677562 101.358695) (width 0.25) (layer "F.Cu") (net 5))
   (segment (start 97.179562 124.472695) (end 95.528562 124.472695) (width 1) (layer "F.Cu") (net 5))
   (segment (start 143.777 85.865) (end 143.777 85.09) (width 0.25) (layer "F.Cu") (net 5))
@@
   (segment (start 134.5 87.847117) (end 134.5 88) (width 0.25) (layer "B.Cu") (net 7))
   (segment (start 138.64076 102.560175) (end 135.152562 99.071977) (width 0.25) (layer "B.Cu") (net 7))
-  (segment (start 149.820562 108.152695) (end 149.820562 103.009695) (width 0.25) (layer "F.Cu") (net 8))
-  (segment (start 150.646562 108.978695) (end 149.820562 108.152695) (width 0.25) (layer "F.Cu") (net 8))
-  (segment (start 152.297562 100.145695) (end 152.297562 101.612695) (width 0.25) (layer "F.Cu") (net 8))
-  (segment (start 150.900562 103.009695) (end 149.820562 103.009695) (width 0.25) (layer "F.Cu") (net 8))
-  (segment (start 150.646562 115.963695) (end 150.646562 108.978695) (width 0.25) (layer "F.Cu") (net 8))
-  (segment (start 152.297562 101.612695) (end 150.900562 103.009695) (width 0.25) (layer "F.Cu") (net 8))
+  (segment (start 152.297562 100.145695) (end 152.297562 102.952438) (width 0.25) (layer "F.Cu") (net 8))
+  (segment (start 150.646562 104.603438) (end 150.646562 115.963695) (width 0.25) (layer "F.Cu") (net 8))
+  (segment (start 152.297562 102.952438) (end 150.646562 104.603438) (width 0.25) (layer "F.Cu") (net 8))
   (segment (start 183.134 112.268) (end 184.531 113.665) (width 0.2) (layer "F.Cu") (net 10))
   (segment (start 184.531 113.665) (end 184.531 119.876133) (width 0.2) (layer "F.Cu") (net 10))

Commit message: Add power-up button
Parts:
- SW1: value SHUTDOWN -> SW_Push; footprint Connector_PinHeader_2.54mm:PinHeader_1x02_P2.54mm_Horizontal -> Button_Switch_THT:SW_PUSH_6mm
- moved SW1 52.2 mm to (192.8, 85.1), turned to 0 degrees
- moved J1 9.68 mm to (197.4, 80.6)
Connections:
- J2 pad 32: unconnected-(J2-Pad32) -> /PWR_EN
- J2 pad 7: /SHUTDOWN -> unconnected-(J2-Pad7)
- R3 pad 1: +BATT -> Net-(R3-Pad1)
- R3 pad 2: Net-(R3-Pad2) -> /PWR_EN
- R4 pad 1: Net-(R3-Pad2) -> /PWR_EN
- SW1 pad 1: /SHUTDOWN -> +BATT
- SW1 pad 2: GND -> Net-(R3-Pad1)
- U5 pad 5: Net-(R3-Pad2) -> /PWR_EN
Routing:
- net Net-(R3-Pad1): track 0.00 -> 18.8 mm
- net /SHUTDOWN: track 16.5 -> 0.00 mm
- net /PWR_EN: track 0.00 -> 13.3 mm
- net GND: track 139.5 -> 126.2 mm, vias 37 -> 38
- net +BATT: track 77.5 -> 66.9 mm, vias 2 -> 1
- net Net-(R3-Pad2): track 6.16 -> 0.00 mm
- net +5V: track 241.8 -> 240.9 mm
Other:
- board text added: "Power On"

Commit message: Use correct footprint for screw terminals
Parts:
- removed J11, J12: Conn_01x02, TerminalBlock_Phoenix:TerminalBlock_Phoenix_PT-1,5-2-5.0-H_1x02_P5.00mm_Horizontal
- added J5: Screw_Terminal_01x04, TerminalBlock_Phoenix:TerminalBlock_Phoenix_MPT-0,5-4-2.54_1x04_P2.54mm_Horizontal, F.Cu at (168.7, 79.5)
Connections:
- net Net-(J11-Pad2) renamed /Pyro Channel Pair/PYRO_A_PWR
- net Net-(J12-Pad2) renamed /Pyro Channel Pair/PYRO_B_PWR
Routing:
- net /Pyro Channel Pair/PYRO_A_PWR: track 30.9 -> 20.7 mm, vias 0 -> 2
- net /Pyro Channel Pair/PYRO_B_PWR: track 3.13 -> 12.5 mm
- net +BATT: track 66.9 -> 60.0 mm
- removed copper zone on F.Cu, net /Pyro Channel Pair/PYRO_A_PWR
- removed copper zone on F.Cu, net /Pyro Channel Pair/PYRO_B_PWR

Commit message: Correct resistor value
Parts:
- R16: value 27k -> 100k
Changed lines of the file:
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@@
       (effects (font (size 1 1) (thickness 0.15)))
     )
-    (fp_text value "27k" (at 0 1.43 90) (layer "F.Fab")
+    (fp_text value "100k" (at 0 1.43 90) (layer "F.Fab")
       (effects (font (size 1 1) (thickness 0.15)))
     )

Commit message: Update servo connector footprints
Parts:
- S0, S1, S2, S3, S4, S5, S6, S7, S8, S9: footprint Connector_PinHeader_2.54mm:PinHeader_1x03_P2.54mm_Vertical -> Connector_PinHeader_2.54mm:PinHeader_1x03_P2.54mm_Horizontal

Commit message: Update version number
Routing:
- net /SDA: track 137.3 -> 136.4 mm
Other:
- board text added: "Raspberry Pi Motherboard V1.1"
- board text removed: "Raspberry Pi Motherboard V1.0"
Changed lines of the file:
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@@
   (gr_line (start 215.289562 79.641695) (end 215.289562 122.821695) (layer "Edge.Cuts") (width 0.1))
   (gr_arc locked (start 79.399562 126.631695) (mid 76.705485 125.515772) (end 75.589562 122.821695) (layer "Edge.Cuts") (width 0.1))
-  (gr_text "Raspberry Pi Motherboard\nV1.0" (at 145.947562 104.279695) (layer "B.SilkS")
+  (gr_text "Raspberry Pi Motherboard\nV1.1" (at 145.947562 104.279695) (layer "B.SilkS")
     (effects (font (size 1 1) (thickness 0.15)) (justify right mirror))
   )
@@
   (via (at 125.378285 87.621715) (size 0.8) (drill 0.4) (layers "F.Cu" "B.Cu") (net 6))
   (via (at 133.25 87.621715) (size 0.8) (drill 0.4) (layers "F.Cu" "B.Cu") (net 6))
-  (segment (start 134.484211 91.265789) (end 134.703042 91.265789) (width 0.25) (layer "B.Cu") (net 6))
+  (segment (start 133.25 87.85) (end 133.25 87.621715) (width 0.25) (layer "B.Cu") (net 6))
   (segment (start 125.378285 87.621715) (end 133.25 87.621715) (width 0.25) (layer "B.Cu") (net 6))
   (segment (start 124.621715 87.621715) (end 125.378285 87.621715) (width 0.25) (layer "B.Cu") (net 6))
   (segment (start 108.127119 87.318) (end 124.318 87.318) (width 0.25) (layer "B.Cu") (net 6))
+  (segment (start 134 91.75) (end 134.703042 92.453042) (width 0.25) (layer "B.Cu") (net 6))
   (segment (start 134.703042 99.258175) (end 138.454562 103.009695) (width 0.25) (layer "B.Cu") (net 6))
   (segment (start 104.169619 91.2755) (end 108.127119 87.318) (width 0.25) (layer "B.Cu") (net 6))
-  (segment (start 133.25 89.812747) (end 133.25 87.621715) (width 0.25) (layer "B.Cu") (net 6))
+  (segment (start 103.251 91.2755) (end 92.121098 91.2755) (width 0.25) (layer "B.Cu") (net 6))
+  (segment (start 147.217562 101.232412) (end 147.217562 100.145695) (width 0.25) (layer "B.Cu") (net 6))
+  (segment (start 134 88.6) (end 133.25 87.85) (width 0.25) (layer "B.Cu") (net 6))
+  (segment (start 92.121098 91.2755) (end 89.729799 93.666799) (width 0.25) (layer "B.Cu") (net 6))
+  (segment (start 145.440279 103.009695) (end 147.217562 101.232412) (width 0.25) (layer "B.Cu") (net 6))
+  (segment (start 103.251 91.2755) (end 104.169619 91.2755) (width 0.25) (layer "B.Cu") (net 6))
+  (segment (start 134 91.75) (end 134 88.6) (width 0.25) (layer "B.Cu") (net 6))
+  (segment (start 134.703042 92.453042) (end 134.703042 99.258175) (width 0.25) (layer "B.Cu") (net 6))
+  (segment (start 124.318 87.318) (end 124.621715 87.621715) (width 0.25) (layer "B.Cu") (net 6))
   (segment (start 138.454562 103.009695) (end 145.440279 103.009695) (width 0.25) (layer "B.Cu") (net 6))
-  (segment (start 103.251 91.2755) (end 92.121098 91.2755) (width 0.25) (layer "B.Cu") (net 6))
-  (segment (start 134.703042 91.265789) (end 134.703042 99.258175) (width 0.25) (layer "B.Cu") (net 6))
-  (segment (start 147.217562 101.232412) (end 147.217562 100.145695) (width 0.25) (layer "B.Cu") (net 6))
-  (segment (start 92.121098 91.2755) (end 89.729799 93.666799) (width 0.25) (layer "B.Cu") (net 6))
-  (segment (start 103.251 91.2755) (end 104.169619 91.2755) (width 0.25) (layer "B.Cu") (net 6))
-  (segment (start 134.703042 91.265789) (end 133.25 89.812747) (width 0.25) (layer "B.Cu") (net 6))
-  (segment (start 145.440279 103.009695) (end 147.217562 101.232412) (width 0.25) (layer "B.Cu") (net 6))
-  (segment (start 134 91.75) (end 134.484211 91.265789) (width 0.25) (layer "B.Cu") (net 6))
-  (segment (start 124.318 87.318) (end 124.621715 87.621715) (width 0.25) (layer "B.Cu") (net 6))
   (segment (start 141.052 89.904) (end 138.096 89.904) (width 0.25) (layer "F.Cu") (net 7))
   (segment (start 122.7864 85.5364) (end 124.118 86.868) (width 0.25) (layer "F.Cu") (net 7))
