File: Motherboard/motherboard_2022_2023/motherboard_2022_2023.kicad_pcb (KiCad board)
At the start: 2 copper layers, 139.7 x 50.8 mm, 67 parts, among them J1 Conn_01x02_Female, J13 Conn_01x22_Shielded, J14 HDMI_C_1.4, J2 Raspberry_Pi_2_3, J3 Conn_02x04_Counter_Clockwise, J4 STEMMA QT, J5 Screw_Terminal_01x04, Q1 AO4838, SW1 SW_Push, U1 XBee_THT, U3 PCA9685PW, U4 MPL3115A2, U5 TPS56424x, U6 SAM-M8Q, U7 MPU-6050, U8 MCP3004

Commit message: Add shutdown switch
Parts:
- added J6: SHUTDOWN, Connector_PinHeader_2.54mm:PinHeader_1x03_P2.54mm_Horizontal, F.Cu at (150.7, 115.7)
Connections:
- J2 pad 7: unconnected-(J2-Pad7) -> /SHUTDOWN
- J5 pad 1: +BATT -> +5V
- J5 pad 3: +BATT -> +5V
Routing:
- net /SHUTDOWN: track 0.00 -> 16.2 mm

Commit message: Add JLCPCB order number placeholder
Other:
- board text added: "Raspberry Pi Motherboard JLCJLCJLCJLC V1.1"
- board text removed: "Raspberry Pi Motherboard V1.1"
Changed lines of the file:
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@@
   (gr_line (start 215.289562 79.641695) (end 215.289562 122.821695) (layer "Edge.Cuts") (width 0.1))
   (gr_arc locked (start 79.399562 126.631695) (mid 76.705485 125.515772) (end 75.589562 122.821695) (layer "Edge.Cuts") (width 0.1))
-  (gr_text "Raspberry Pi Motherboard\nV1.1" (at 145.947562 104.279695) (layer "B.SilkS")
+  (gr_text "Raspberry Pi Motherboard\nJLCJLCJLCJLC V1.1" (at 145.947562 104.279695) (layer "B.SilkS")
     (effects (font (size 1 1) (thickness 0.15)) (justify right mirror))
   )

Commit message: Delete SAM-M8Q, switch high-current to 5V
Parts:
- removed TP1: RX, TestPoint:TestPoint_Pad_D1.0mm
- removed TP2: TX, TestPoint:TestPoint_Pad_D1.0mm
- removed U6: SAM-M8Q, RF_GPS:ublox_SAM-M8Q
Routing:
- net /PPS: track 78.7 -> 0.00 mm
- net +BATT: track 60.0 -> 25.1 mm
- net +3V3: track 256.2 -> 223.2 mm
- net GND: track 126.2 -> 102.7 mm, vias 38 -> 29
- net /SDA: track 136.4 -> 113.8 mm, vias 5 -> 4
- net +5V: track 240.9 -> 261.9 mm
- net /SCL: track 133.0 -> 115.0 mm, vias 5 -> 4
- net Net-(TP2-Pad1): track 3.94 -> 0.00 mm
- net Net-(TP1-Pad1): track 3.94 -> 0.00 mm

Commit message: Organize schematics
Parts:
- J1: value Conn_01x02_Female -> POWER
- J3: value Conn_02x04_Counter_Clockwise -> IO Expansion
- S0, S1, S2, S3, S4, S5, S6, S7, S8, S9: value Conn_01x03_Male -> Servo Port
Connections:
- J2 pad 16: /PPS -> unconnected-(J2-Pad16)

Commit message: Start adding selectable i2c bus to board
Parts:
- added JP3: SolderJumper_2_Open, Jumper:SolderJumper-2_P1.3mm_Open_RoundedPad1.0x1.5mm, F.Cu at (143.3, 107.2)
- added JP4: SolderJumper_2_Open, Jumper:SolderJumper-2_P1.3mm_Open_RoundedPad1.0x1.5mm, F.Cu at (143.3, 111.3)
- added JP5: SolderJumper_2_Open, Jumper:SolderJumper-2_P1.3mm_Open_RoundedPad1.0x1.5mm, F.Cu at (145.8, 107.2)
- added JP7: SolderJumper_2_Open, Jumper:SolderJumper-2_P1.3mm_Open_RoundedPad1.0x1.5mm, F.Cu at (147.3, 135.3)
- added JP8: SolderJumper_2_Open, Jumper:SolderJumper-2_P1.3mm_Open_RoundedPad1.0x1.5mm, F.Cu at (154.2, 135.9)
- added JPe: SolderJumper_2_Open, Jumper:SolderJumper-2_P1.3mm_Open_RoundedPad1.0x1.5mm, F.Cu at (145.8, 111.3)
Connections:
- J2 pad 12: unconnected-(J2-Pad12) -> /Buzzer
- J2 pad 27: unconnected-(J2-Pad27) -> /SDA_HW_0
- J2 pad 28: unconnected-(J2-Pad28) -> /SCL_HW_0
- J2 pad 3: /SDA -> /SDA_HW_1
- J2 pad 33: /Buzzer -> unconnected-(J2-Pad33)
- J2 pad 5: /SCL -> /SCL_HW_1
Routing:
- net /Buzzer: track 88.8 -> 53.0 mm, vias 1 -> 0
- net /SCL_HW_1: track 0.00 -> 20.8 mm
- net /SDA_HW_1: track 0.00 -> 8.03 mm
- net +3V3: track 223.2 -> 220.5 mm
- net +BATT: track 25.1 -> 26.7 mm
- net /SCL: track 115.0 -> 113.8 mm, vias 4 -> 5
- net /SDA: track 113.8 -> 114.0 mm, vias 4 -> 5
- net GND: vias 29 -> 31

Commit message: Lots of adjustments, 3 way I2C bus selection, SMD diodes
Parts:
- removed JPe: SolderJumper_2_Open, Jumper:SolderJumper-2_P1.3mm_Open_RoundedPad1.0x1.5mm
- added JP6: SolderJumper_2_Open, Jumper:SolderJumper-2_P1.3mm_Open_RoundedPad1.0x1.5mm, F.Cu at (145.8, 111.3)
- added R1: 10k, Resistor_SMD:R_0603_1608Metric, F.Cu at (139.3, 108.1)
- added R2: 10k, Resistor_SMD:R_0603_1608Metric, F.Cu at (139.3, 110.0)
- D1, D2: footprint Diode_THT:D_DO-41_SOD81_P2.54mm_Vertical_AnodeUp -> Diode_SMD:D_SOD-323_HandSoldering
- moved BZ1 53.1 mm to (154.7, 83.3), turned to -135 degrees
- moved JP7 28.2 mm to (148.3, 107.2), turned to 90 degrees
- moved JP8 25.4 mm to (148.3, 111.3), turned to 90 degrees
- moved R10 4.34 mm to (175.1, 91.9)
- moved JP1 4.34 mm to (176.8, 88.8)
- moved R9 4.34 mm to (176.8, 91.9)
- moved D1 3.85 mm to (178.6, 92.6), turned to 90 degrees
- moved J5 3.24 mm to (172.0, 79.5)
- moved D2 2.90 mm to (173.4, 92.6), turned to 90 degrees
- moved R12 2.87 mm to (169.8, 91.9)
- moved JP2 2.87 mm to (171.6, 88.8)
- moved R11 2.87 mm to (171.6, 91.9)
- moved R14 2.05 mm to (164.1, 93.6)
- moved R7 2.05 mm to (162.2, 93.6)
- moved R8 2.05 mm to (165.9, 93.6)
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Connections:
- J2 pad 11: unconnected-(J2-Pad11) -> /SDA_SW
- J2 pad 13: unconnected-(J2-Pad13) -> /SCL_SW
Routing:
- net /SCL_HW_0: track 0.00 -> 48.5 mm, vias 0 -> 1
- net /SDA_HW_0: track 0.00 -> 43.4 mm, vias 0 -> 1
- net /Buzzer: track 53.0 -> 13.8 mm
- net /SCL_SW: track 0.00 -> 18.9 mm
- net /SDA_SW: track 0.00 -> 12.6 mm
- net GND: track 102.7 -> 108.5 mm
- net /SCL: track 113.8 -> 118.0 mm, vias 5 -> 4
- net /PWM_2: track 91.7 -> 95.2 mm
- net /PWM_1: track 101.6 -> 104.6 mm
- net /PWM_0: track 105.1 -> 108.1 mm
- net +5V: track 261.9 -> 259.2 mm
- net /Pyro Channel Pair/PYRO_A_PWR: track 20.7 -> 23.3 mm
- net /XBEE_UART_TX: track 29.5 -> 32.1 mm
- net /PYRO_B: track 37.3 -> 39.4 mm
- net /PYRO_A: track 33.2 -> 35.2 mm
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Other:
- outline, holes or cut-outs redrawn
- board text added: "HW0"
- board text added: "HW1"
- board text added: "SW"

Commit message: Add jumper to select pyro voltage
Parts:
- added JP9: PYRO_V, Jumper:SolderJumper-3_P2.0mm_Open_TrianglePad1.0x1.5mm, F.Cu at (175.6, 79.2)
- moved C12 0.56 mm to (118.0, 87.4)
Connections:
- J2 pad 18: /GPIO_1 -> unconnected-(J2-Pad18)
- J2 pad 21: unconnected-(J2-Pad21) -> /GPIO_1
- J2 pad 22: /GPIO_2 -> unconnected-(J2-Pad22)
- J2 pad 23: unconnected-(J2-Pad23) -> /GPIO_2
- J5 pad 1: +5V -> /Pyro Channel Pair/V_BAT
- J5 pad 3: +5V -> /Pyro Channel Pair/V_BAT
Routing:
- net +BATT: track 26.7 -> 44.9 mm
- net +5V: track 259.2 -> 243.9 mm
- net /Pyro Channel Pair/V_BAT: track 0.00 -> 12.0 mm
- net /GPIO_1: track 35.8 -> 29.0 mm
- net /GPIO_2: track 28.6 -> 24.2 mm
- net GND: track 108.5 -> 108.1 mm, vias 31 -> 33
Other:
- board text added: "5V"
- board text added: "BAT"
- board text added: "Pyro Voltage"

Commit message: Shrunk PCB :)
Parts:
- moved J4 36.7 mm to (107.3, 87.3)
- moved S8 33.6 mm to (107.3, 107.6)
- moved S9 32.6 mm to (107.3, 116.5)
- moved S7 28.9 mm to (107.3, 98.7), turned to 180 degrees
- moved H1 27.9 mm to (107.3, 79.6), turned to 90 degrees
- moved H3 27.9 mm to (107.3, 122.8)
- moved S6 16.3 mm to (113.7, 79.6)
- moved S5 14.1 mm to (122.6, 79.6)
- moved S4 12.7 mm to (132.7, 79.6)
- moved C15 11.2 mm to (205.6, 94.0), turned to 180 degrees
- moved U8 10.8 mm to (206.4, 87.5), turned to -90 degrees
- moved R16 10.2 mm to (203.9, 82.2)
- moved R17 10.1 mm to (205.8, 82.2)
- moved S3 8.97 mm to (141.6, 79.6)
- moved S2 8.51 mm to (208.9, 93.6)
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Connections:
- U3 pad 13: /PWM_7 -> unconnected-(U3-Pad13)
- U3 pad 15: /PWM_8 -> /PWM_7
- U3 pad 16: /PWM_9 -> /PWM_8
- U3 pad 17: unconnected-(U3-Pad17) -> /PWM_9
Routing:
- net /SDA: track 115.9 -> 72.6 mm, vias 5 -> 4
- net /SCL: track 118.0 -> 75.2 mm, vias 4 -> 3
- net +3V3: track 220.2 -> 184.6 mm
- net /PWM_8: track 54.3 -> 28.8 mm
- net /PWM_9: track 57.3 -> 38.0 mm
- net /PWM_7: track 40.9 -> 22.9 mm
- net /PWM_6: track 30.7 -> 13.5 mm
- net /PWM_5: track 20.4 -> 5.58 mm
- net +5V: track 243.9 -> 253.7 mm
- net /PWM_3: track 9.97 -> 18.0 mm, vias 0 -> 1
- net /PWM_1: track 104.6 -> 97.7 mm, vias 2 -> 1
- net /SCLK: track 13.9 -> 17.7 mm
- net Net-(R16-Pad1): track 11.5 -> 7.84 mm
- net +BATT: track 44.9 -> 41.7 mm
- net /PWM_0: track 108.1 -> 105.1 mm, vias 2 -> 1
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Other:
- board size 139.7 x 50.8 mm -> 109.2 x 50.8 mm
- board text removed: "hi mom"
