File: Motherboard/motherboard_2022_2023/motherboard_2022_2023.kicad_pcb (KiCad board)
At the start: 2 copper layers, 109.2 x 50.8 mm, 74 parts, among them J1 POWER, J13 Conn_01x22_Shielded, J14 HDMI_C_1.4, J2 Raspberry_Pi_2_3, J3 IO Expansion, J4 STEMMA QT, J5 Screw_Terminal_01x04, J6 SHUTDOWN, Q1 AO4838, SW1 SW_Push, U1 XBee_THT, U3 PCA9685PW, U4 MPL3115A2, U5 TPS56424x, U7 MPU-6050, U8 MCP3004

Commit message: Disconnect XBee from SPI bus (no longer needed)
Connections:
- J2 pad 11: /XBEE_CS -> /XBEE_RESET
- J2 pad 37: /XBEE_INT -> unconnected-(J2-Pad37)
- U1 pad 11: /MOSI -> unconnected-(U1-Pad11)
- U1 pad 17: /XBEE_CS -> unconnected-(U1-Pad17)
- U1 pad 18: /SCLK -> unconnected-(U1-Pad18)
- U1 pad 19: /XBEE_INT -> unconnected-(U1-Pad19)
- U1 pad 4: /MISO -> unconnected-(U1-Pad4)
- U1 pad 5: unconnected-(U1-Pad5) -> /XBEE_RESET
Routing:
- net /SCLK: track 115.3 -> 17.7 mm
- net /MOSI: track 114.7 -> 17.4 mm
- net /XBEE_INT: track 89.0 -> 0.00 mm
- net /MISO: track 87.0 -> 23.0 mm, vias 1 -> 0
- net /XBEE_CS: track 55.4 -> 0.00 mm
- net /XBEE_RESET: track 0.00 -> 38.7 mm
- net /XBEE_UART_~{CTS}: track 78.5 -> 72.7 mm

Commit message: Tune differential pair lengths
Routing:
- net /HDMI CSI Conversion/D1-: track 19.9 -> 20.5 mm
- net /HDMI CSI Conversion/DC-: track 17.9 -> 18.5 mm
- net /HDMI CSI Conversion/D0-: track 21.9 -> 22.5 mm
- net +BATT: track 41.2 -> 41.3 mm, vias 1 -> 0

Commit message: Added RGB Indicator LED and Potential Candidates
Parts:
- added D3: RED, LED_SMD:LED_1206_3216Metric, F.Cu at (134.0, 124.1)
- added D4: LED_RGBA, LED_SMD:LED_RGB_1210, F.Cu at (121.2, 103.2)
- added R13: 120, Resistor_SMD:R_0603_1608Metric, F.Cu at (129.4, 124.1)
- added R18: 180, Resistor_SMD:R_0603_1608Metric, F.Cu at (123.7, 98.1)
- added R19: 180, Resistor_SMD:R_0603_1608Metric, F.Cu at (121.2, 98.1)
- added R20: 120, Resistor_SMD:R_0603_1608Metric, F.Cu at (118.6, 98.1)
Connections:
- U3 pad 18: unconnected-(U3-Pad18) -> /LED_R
- U3 pad 19: unconnected-(U3-Pad19) -> /LED_G
- U3 pad 20: unconnected-(U3-Pad20) -> /LED_B
Routing:
- net GND: vias 33 -> 32

Commit message: Update GPIO silkscreen
Other:
- board text added: "IO 3V3 3V3 G05 G11 G06 G13 GND GND"
- board text removed: "IO 3V3 3V3 I25 I24 I06 I26 GND GND"
Changed lines of the file:
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@@
     (effects (font (size 1 1) (thickness 0.15)) (justify right mirror))
   )
-  (gr_text "IO\n3V3 3V3\nI25 I24\nI06 I26\nGND GND" (at 185.674 117.094 90) (layer "B.SilkS")
+  (gr_text "IO\n3V3 3V3\nG05 G11\nG06 G13\nGND GND" (at 185.674 117.094 90) (layer "B.SilkS")
     (effects (font (size 1.778 1.5) (thickness 0.3)) (justify right mirror))
   )

Commit message: Traced New RGB LED
Parts:
- D4: footprint LED_SMD:LED_RGB_1210 -> custom-footprints:B3213GBR
- R18, R19: value 180 -> 120
- R20: value 120 -> 82
- moved D4 20.6 mm to (115.1, 83.6), turned to 180 degrees
- moved D3 19.7 mm to (114.3, 124.5)
- moved R13 16.7 mm to (131.0, 107.5), turned to 90 degrees
- moved R18 9.34 mm to (132.6, 95.3)
- moved R19 9.34 mm to (130.1, 95.3)
- moved R20 9.34 mm to (127.5, 95.3)
- moved J4 0.62 mm to (107.3, 87.9)
Routing:
- net Net-(D4-Pad3): track 0.00 -> 30.5 mm, vias 0 -> 2
- net Net-(D4-Pad2): track 0.00 -> 27.2 mm, vias 0 -> 2
- net Net-(D3-Pad1): track 0.00 -> 26.2 mm
- net Net-(D3-Pad2): track 0.00 -> 25.0 mm
- net Net-(D4-Pad1): track 0.00 -> 24.3 mm, vias 0 -> 2
- net /LED_R: track 0.00 -> 5.48 mm
- net /LED_B: track 0.00 -> 5.03 mm
- net /LED_G: track 0.00 -> 4.70 mm
- net +3V3: track 191.0 -> 192.9 mm
- net /SDA: track 72.6 -> 73.4 mm
- net /SCL: track 75.2 -> 75.9 mm
- net GND: vias 32 -> 34

Commit message: Trace Fixed
Other:
- board text added: "IO 3V3 3V3 I25 I24 I06 I26 GND GND"
- board text removed: "IO 3V3 3V3 G05 G11 G06 G13 GND GND"
Changed lines of the file:
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@@
     (effects (font (size 1 1) (thickness 0.15)) (justify right mirror))
   )
-  (gr_text "IO\n3V3 3V3\nG05 G11\nG06 G13\nGND GND" (at 185.674 117.094 90) (layer "B.SilkS")
+  (gr_text "IO\n3V3 3V3\nI25 I24\nI06 I26\nGND GND" (at 185.674 117.094 90) (layer "B.SilkS")
     (effects (font (size 1.778 1.5) (thickness 0.3)) (justify right mirror))
   )

Commit message: Simplify LED routing
Parts:
- moved R13 8.08 mm to (126.9, 114.4), turned to -135 degrees
Connections:
- D3 pad 1: Net-(D3-Pad1) -> GND
- R13 pad 1: Net-(D3-Pad1) -> Net-(U1-Pad6)
- R13 pad 2: GND -> Net-(D3-Pad2)
- U1 pad 6: Net-(D3-Pad2) -> Net-(U1-Pad6)
Routing:
- net Net-(D3-Pad1): track 26.2 -> 0.00 mm
- net Net-(D3-Pad2): track 25.0 -> 14.5 mm
- net Net-(U1-Pad6): track 0.00 -> 8.86 mm
Changed lines of the file:
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@@
   (net 49 "/PWM_8")
   (net 50 "unconnected-(U3-Pad13)")
-  (net 51 "Net-(D3-Pad1)")
+  (net 51 "Net-(U1-Pad6)")
   (net 52 "Net-(D4-Pad1)")
   (net 53 "Net-(D4-Pad2)")
@@
   )
   (footprint "Resistor_SMD:R_0603_1608Metric" (layer "F.Cu")
-    (at 131.035 107.502742 90)
+    (at 126.873 114.427 -135)
     (descr "Resistor SMD 0603 (1608 Metric), square (rectangular) end terminal, IPC_7351 nominal, (Body size source: IPC-SM-782 page 72, https://www.pcb-3d.com/wordpress/wp-content/uploads/ipc-sm-782a_amendment_1_and_2.pdf), generated with kicad-footprint-generator")
     (tags "resistor")
@@
     (property "Sheetname" "")
     (attr smd)
-    (fp_text reference "R13" (at 0 -1.43 90) (layer "F.SilkS")
+    (fp_text reference "R13" (at 0 -1.43 45) (layer "F.SilkS")
       (effects (font (size 1 1) (thickness 0.15)))
     )
-    (fp_text value "120" (at 0 1.43 90) (layer "F.Fab")
+    (fp_text value "120" (at 0 1.43 45) (layer "F.Fab")
       (effects (font (size 1 1) (thickness 0.15)))
     )
-    (fp_text user "${REFERENCE}" (at 0 0 90) (layer "F.Fab")
+    (fp_text user "${REFERENCE}" (at 0 0 45) (layer "F.Fab")
       (effects (font (size 0.4 0.4) (thickness 0.06)))
     )
@@
     (fp_line (start -0.8 -0.4125) (end 0.8 -0.4125) (layer "F.Fab") (width 0.1))
     (fp_line (start 0.8 -0.4125) (end 0.8 0.4125) (layer "F.Fab") (width 0.1))
-    (pad "1" smd roundrect (at -0.825 0 90) (size 0.8 0.95) (layers "F.Cu" "F.Paste" "F.Mask") (roundrect_rratio 0.25)
-      (net 51 "Net-(D3-Pad1)") (pintype "passive"))
-    (pad "2" smd roundrect (at 0.825 0 90) (size 0.8 0.95) (layers "F.Cu" "F.Paste" "F.Mask") (roundrect_rratio 0.25)
-      (net 2 "GND") (pintype "passive"))
+    (pad "1" smd roundrect (at -0.825 0 225) (size 0.8 0.95) (layers "F.Cu" "F.Paste" "F.Mask") (roundrect_rratio 0.25)
+      (net 51 "Net-(U1-Pad6)") (pintype "passive"))
+    (pad "2" smd roundrect (at 0.825 0 225) (size 0.8 0.95) (layers "F.Cu" "F.Paste" "F.Mask") (roundrect_rratio 0.25)
+      (net 46 "Net-(D3-Pad2)") (pintype "passive"))
     (model "${KICAD6_3DMODEL_DIR}/Resistor_SMD.3dshapes/R_0603_1608Metric.wrl"
       (offset (xyz 0 0 0))
@@
     (fp_line (start -1.6 0.8) (end 1.6 0.8) (layer "F.Fab") (width 0.1))
     (pad "1" smd roundrect (at -1.4 0) (size 1.25 1.75) (layers "F.Cu" "F.Paste" "F.Mask") (roundrect_rratio 0.2)
-      (net 51 "Net-(D3-Pad1)") (pinfunction "K") (pintype "passive"))
+      (net 2 "GND") (pinfunction "K") (pintype "passive"))
     (pad "2" smd roundrect (at 1.4 0) (size 1.25 1.75) (layers "F.Cu" "F.Paste" "F.Mask") (roundrect_rratio 0.2)
       (net 46 "Net-(D3-Pad2)") (pinfunction "A") (pintype "passive"))
@@
       (net 35 "/XBEE_RESET") (pinfunction "~{RESET}") (pintype "input"))
     (pad "6" thru_hole circle (at 22 -10 90) (size 1.35 1.35) (drill 0.8) (layers *.Cu *.Mask)
-      (net 46 "Net-(D3-Pad2)") (pinfunction "DIO10/PWM0/RSSI_PWM") (pintype "bidirectional"))
+      (net 51 "Net-(U1-Pad6)") (pinfunction "DIO10/PWM0/RSSI_PWM") (pintype "bidirectional"))
     (pad "7" thru_hole circle (at 22 -12 90) (size 1.35 1.35) (drill 0.8) (layers *.Cu *.Mask)
       (net 36 "unconnected-(U1-Pad7)") (pinfunction "DIO11/PWM1") (pintype "bidirectional+no_connect"))
@@
   (segment (start 133.206562 89.264562) (end 132.461 88.519) (width 0.25) (layer "F.Cu") (net 2))
   (segment (start 207.6696 91.7067) (end 206.3996 92.9767) (width 0.25) (layer "F.Cu") (net 2))
+  (segment (start 112.9 124.46) (end 112.9 124.336) (width 0.2) (layer "F.Cu") (net 2))
   (segment (start 168.447062 89.039695) (end 168.638062 89.230695) (width 0.25) (layer "F.Cu") (net 2))
   (segment (start 147.803 90.208) (end 147.8725 90.208) (width 0.25) (layer "F.Cu") (net 2))
@@
   (segment (start 143.082 109.660097) (end 136.017 116.725097) (width 0.25) (layer "B.Cu") (net 39))
   (segment (start 134.491604 119.38) (end 131.710905 119.38) (width 0.25) (layer "B.Cu") (net 39))
-  (segment (start 117.660257 124.46) (end 115.7 124.46) (width 0.2) (layer "F.Cu") (net 46))
-  (segment (start 133.960562 108.159695) (end 117.660257 124.46) (width 0.2) (layer "F.Cu") (net 46))
+  (segment (start 116.84 124.46) (end 115.7 124.46) (width 0.25) (layer "F.Cu") (net 46))
+  (segment (start 126.289637 115.010363) (end 116.84 124.46) (width 0.25) (layer "F.Cu") (net 46))
   (segment (start 129.306562 91.006424) (end 129.306562 89.997195) (width 0.2) (layer "F.Cu") (net 48))
   (segment (start 109.7716 108.9597) (end 109.7716 97.7837) (width 0.2) (layer "F.Cu") (net 48))
@@
   (segment (start 126.0276 93.7197) (end 113.269915 93.7197) (width 0.2) (layer "F.Cu") (net 49))
   (segment (start 109.3716 100.4697) (end 107.3396 102.5017) (width 0.2) (layer "F.Cu") (net 49))
-  (segment (start 112.9 124.46) (end 112.9 124.336) (width 0.2) (layer "F.Cu") (net 51))
-  (segment (start 131.035 110.519571) (end 131.035 108.327742) (width 0.2) (layer "F.Cu") (net 51))
-  (segment (start 114.3 122.936) (end 118.618571 122.936) (width 0.2) (layer "F.Cu") (net 51))
-  (segment (start 112.9 124.336) (end 114.3 122.936) (width 0.2) (layer "F.Cu") (net 51))
-  (segment (start 118.618571 122.936) (end 131.035 110.519571) (width 0.2) (layer "F.Cu") (net 51))
+  (segment (start 133.140305 108.159695) (end 133.960562 108.159695) (width 0.25) (layer "F.Cu") (net 51))
+  (segment (start 127.456363 113.843637) (end 133.140305 108.159695) (width 0.25) (layer "F.Cu") (net 51))
   (segment (start 114.808 95.504) (end 118.238396 95.504) (width 0.25) (layer "F.Cu") (net 52))
   (segment (start 127.762 96.397258) (end 127.762 96.361758) (width 0.25) (layer "F.Cu") (net 52))

Commit message: Update LEDs
Parts:
- added D5: RED, LED_SMD:LED_0603_1608Metric, F.Cu at (112.6, 83.1)
- added R21: 560, Resistor_SMD:R_0603_1608Metric, F.Cu at (114.6, 83.0)
- D3: footprint LED_SMD:LED_1206_3216Metric -> LED_SMD:LED_0603_1608Metric
- D4: footprint custom-footprints:B3213GBR -> LED_SMD:LED_RGB_5050-6
- R13: value 120 -> 68
- R18, R19: value 120 -> 15
- R20: value 82 -> 68
- moved D4 4.84 mm to (113.9, 88.3), turned to -90 degrees
- moved D3 1.30 mm to (113.0, 124.7)
- moved R18 0.65 mm to (132.0, 95.3)
- moved R20 0.62 mm to (128.1, 95.3)
Connections:
- D4 pad 1: Net-(D4-Pad1) -> +3V3
- D4 pad 2: Net-(D4-Pad2) -> +3V3
- D4 pad 3: Net-(D4-Pad3) -> +3V3
- D4 pad 4: +3V3 -> Net-(D4-Pad4)
- R18 pad 2: Net-(D4-Pad3) -> Net-(D4-Pad4)
- R19 pad 2: Net-(D4-Pad2) -> Net-(D4-Pad5)
- R20 pad 2: Net-(D4-Pad1) -> Net-(D4-Pad6)
Routing:
- net Net-(D4-Pad3): track 30.5 -> 0.00 mm, vias 2 -> 0
- net Net-(D4-Pad2): track 27.2 -> 0.00 mm, vias 2 -> 0
- net Net-(D4-Pad4): track 0.00 -> 25.7 mm, vias 0 -> 2
- net Net-(D4-Pad1): track 24.3 -> 0.00 mm, vias 2 -> 0
- net Net-(D4-Pad5): track 0.00 -> 22.1 mm, vias 0 -> 2
- net Net-(D4-Pad6): track 0.00 -> 18.7 mm, vias 0 -> 2
- net +5V: track 68.9 -> 72.4 mm
- net Net-(D3-Pad2): track 14.5 -> 16.5 mm
- net Net-(D5-Pad2): track 0.00 -> 1.91 mm
- net +3V3: track 192.9 -> 191.0 mm
- net /SDA_HW_0: track 43.4 -> 42.1 mm
- net /SCL_HW_0: track 48.5 -> 47.2 mm
Other:
- board text removed: "STEMMA QT I2C"
