File: Motherboard/motherboard_2022_2023/buck.kicad_sch (KiCad schematic)
At the start: 12 parts, among them SW1 SW_Push, U5 TPS56424x

Commit message: Change button footprint
Parts:
- SW1: footprint Button_Switch_THT:SW_PUSH_6mm -> custom-footprints:SW_PUSH_6mm_2pin
Changed lines of the file:
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@@
     (property "Reference" "SW1" (id 0) (at 72.39 36.83 0))
     (property "Value" "SW_Push" (id 1) (at 72.39 39.37 0))
-    (property "Footprint" "Button_Switch_THT:SW_PUSH_6mm" (id 2) (at 72.39 29.21 0)
+    (property "Footprint" "custom-footprints:SW_PUSH_6mm_2pin" (id 2) (at 72.39 29.21 0)
       (effects (font (size 1.27 1.27)) hide)
     )
