File: Motherboard/motherboard_2022_2023/buck.kicad_sch (KiCad schematic)
At the start: 12 parts, among them SW1 SW_Push, U5 TPS56424x

Commit message: Revert "Change button footprint"
This reverts commit 62573433dc6a31f4ca51f9e5dc16294e81f44105.
Parts:
- SW1: footprint custom-footprints:SW_PUSH_6mm_2pin -> Button_Switch_THT:SW_PUSH_6mm
Changed lines of the file:
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@@
     (property "Reference" "SW1" (id 0) (at 72.39 36.83 0))
     (property "Value" "SW_Push" (id 1) (at 72.39 39.37 0))
-    (property "Footprint" "custom-footprints:SW_PUSH_6mm_2pin" (id 2) (at 72.39 29.21 0)
+    (property "Footprint" "Button_Switch_THT:SW_PUSH_6mm" (id 2) (at 72.39 29.21 0)
       (effects (font (size 1.27 1.27)) hide)
     )

Commit message: Fixed LED
Parts:
- C5: value 100nF -> 100n
Changed lines of the file:
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@@
       (effects (font (size 1.27 1.27)) (justify left))
     )
-    (property "Value" "100nF" (id 1) (at 201.93 43.1799 0)
+    (property "Value" "100n" (id 1) (at 201.93 43.1799 0)
       (effects (font (size 1.27 1.27)) (justify left))
     )
